File: gpio.kicad_sch (KiCad schematic)
At the start: 0 parts

Commit message: Added 12V GPIO module
Parts:
- added Q1, Q2, Q3, Q4: AUIRF7316QTR, Package_SO:SO-8_3.9x4.9mm_P1.27mm, symbol symbols:AUIRF7316QTR
- added R10, R11, R12, R13, R14, R15, R16, R17, R18, R19, R20, R21, R22, R23, R24, R25, R26, R27, R28, R29, R6, R7, R8, R9: R, symbol Device:R
- added U4: NPIC6C596ADJ, Package_SO:SOIC-16_4.55x10.3mm_P1.27mm, symbol Custom-Symbols:NPIC6C596ADJ
- added U5: PCF8574DWR, symbol symbols:PCF8574DWR
Connections:
- new net +12V: Q1.1 (S), Q1.3 (S), Q2.1 (S), Q2.3 (S), Q3.1 (S), Q3.3 (S), Q4.1 (S), Q4.3 (S), R22.1, R23.1, R24.1, R25.1, R26.1, R27.1, R28.1, R29.1
- new net +3V3: U4.1 (Vcc), U5.16 (Vcc)
- new net DS: U4.2 (DS)
- new net GND: R11.2, R13.2, R15.2, R17.2, R19.2, R21.2, R7.2, R9.2, U4.16 (GND), U5.1 (A0), U5.2 (A1), U5.3 (A2), U5.8 (GND)
- new net I_{1}: R6.2, R7.1, U5.4 (P0)
- new net I_{2}: R8.2, R9.1, U5.5 (P1)
- new net I_{3}: R10.2, R11.1, U5.6 (P2)
- new net I_{4}: R12.2, R13.1, U5.7 (P3)
- new net I_{5}: R14.2, R15.1, U5.12 (P7)
- new net I_{6}: R16.2, R17.1, U5.11 (P6)
- new net I_{7}: R18.2, R19.1, U5.10 (P5)
- new net I_{8}: R20.2, R21.1, U5.9 (P4)
- new net Input_{1}: R6.1
- new net Input_{2}: R8.1
- new net Input_{3}: R10.1
- new net Input_{4}: R12.1
- new net Input_{5}: R14.1
- new net Input_{6}: R16.1
- new net Input_{7}: R18.1
- new net Input_{8}: R20.1
- new net OUT_CTL_{1}: Q1.2 (G), R22.2, U4.3 (Q0)
- new net OUT_CTL_{2}: Q1.4 (G), R23.2, U4.4 (Q1)
- new net OUT_CTL_{3}: Q2.2 (G), R24.2, U4.5 (Q2)
- new net OUT_CTL_{4}: Q2.4 (G), R25.2, U4.6 (Q3)
- new net OUT_CTL_{5}: Q3.2 (G), R26.2, U4.11 (Q4)
- new net OUT_CTL_{6}: Q3.4 (G), R27.2, U4.12 (Q5)
- new net OUT_CTL_{7}: Q4.2 (G), R28.2, U4.13 (Q6)
- new net OUT_CTL_{8}: Q4.4 (G), R29.2, U4.14 (Q7)
- new net OUT_{1}: Q1.6 (D), Q1.7 (D)
- new net OUT_{2}: Q1.5 (D), Q1.8 (D)
- new net OUT_{3}: Q2.6 (D), Q2.7 (D)
- new net OUT_{4}: Q2.5 (D), Q2.8 (D)
- new net OUT_{5}: Q3.6 (D), Q3.7 (D)
- new net OUT_{6}: Q3.5 (D), Q3.8 (D)
- new net OUT_{7}: Q4.6 (D), Q4.7 (D)
- new net OUT_{8}: Q4.5 (D), Q4.8 (D)
- new net SCL: U5.14 (SCL)
- new net SDA: U5.15 (SDA)
- new net SHCP: U4.15 (SHCP)
- new net STCP: U4.10 (STCP)
- new net ~INT: U5.13 (~INT)
- new net ~MR: U4.7 (~MR)
- new net ~OE: U4.8 (~OE)
- no-connect marks 0 -> 1
Other:
- note added: "An I2C IO expander is used to read the inputs instead of connecting to the pi's gpio pins directly. This is mainly done for insurance so that the pi's pins cannot be accidentally exposed to the 12V signal."
- note added: "NOTE: By far the most common use for these inputs will be to read the value of switches. Need to think more about the best way to achieve this, it is most likely not this. It might be nice to combine Input and Output pins into a single circuit which can be configured in software to act like either, like the gpio modules on microprocessors. Perhaps a "switch detection" mode could be added as well,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"
- note added: "Voltage Divider Network (12V -> 5V) Used to read 12V digital input signals from other parts of the bike Use integrated resistor network if possible (TODO: spec)"
