File: power.kicad_sch (KiCad schematic)
At the start: 13 parts, among them J5 Barrel_Jack, U3 AP64501

Commit message: Adding footprints and step files for connectors
Parts:
- C5: renamed from C4; value 60uF@12V -> C
- C7: renamed from C5; value 100nF -> C; footprint (none) -> Capacitor_SMD:C_0805_2012Metric
- C9: renamed from C8; value 140uF@5V -> C
- L1: value 3.3uH@5A -> 3.3uH
Changed lines of the file:
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@@
     (in_bom yes) (on_board yes)
     (property "Reference" "L1" (id 0) (at 158.75 53.702 90))
-    (property "Value" "3.3uH@5A" (id 1) (at 161.29 49.651 90))
+    (property "Value" "3.3uH" (id 1) (at 161.29 49.651 90))
     (property "Footprint" "" (id 2) (at 158.75 52.07 0)
       (effects (font (size 1.27 1.27)) hide)
@@
   (symbol (lib_id "Device:C") (at 105.41 60.96 0) (unit 1)
     (in_bom yes) (on_board yes)
-    (property "Reference" "C4" (id 0) (at 108.3311 59.8106 0)
-      (effects (font (size 1.27 1.27)) (justify left))
-    )
-    (property "Value" "60uF@12V" (id 1) (at 91.821 60.839 0)
+    (property "Reference" "C5" (id 0) (at 108.3311 59.8106 0)
+      (effects (font (size 1.27 1.27)) (justify left))
+    )
+    (property "Value" "C" (id 1) (at 91.821 60.839 0)
       (effects (font (size 1.27 1.27)) (justify left))
     )
@@
   (symbol (lib_id "Device:C") (at 116.84 60.96 0) (unit 1)
     (in_bom yes) (on_board yes)
-    (property "Reference" "C5" (id 0) (at 119.7611 59.8106 0)
-      (effects (font (size 1.27 1.27)) (justify left))
-    )
-    (property "Value" "100nF" (id 1) (at 117.221 63.379 0)
-      (effects (font (size 1.27 1.27)) (justify left))
-    )
-    (property "Footprint" "" (id 2) (at 117.8052 64.77 0)
+    (property "Reference" "C7" (id 0) (at 119.7611 59.8106 0)
+      (effects (font (size 1.27 1.27)) (justify left))
+    )
+    (property "Value" "C" (id 1) (at 117.221 63.379 0)
+      (effects (font (size 1.27 1.27)) (justify left))
+    )
+    (property "Footprint" "Capacitor_SMD:C_0805_2012Metric" (id 2) (at 117.8052 64.77 0)
       (effects (font (size 1.27 1.27)) hide)
     )
@@
   (symbol (lib_id "Device:C") (at 168.91 60.96 0) (unit 1)
     (in_bom yes) (on_board yes)
-    (property "Reference" "C8" (id 0) (at 171.8311 59.8106 0)
-      (effects (font (size 1.27 1.27)) (justify left))
-    )
-    (property "Value" "140uF@5V" (id 1) (at 171.831 62.109 0)
-      (effects (font (size 1.27 1.27)) (justify left))
-    )
+    (property "Reference" "C9" (id 0) (at 171.8311 59.8106 0)
+      (effects (font (size 1.27 1.27)) (justify left))
+    )
+    (property "Value" "C" (id 1) (at 171.831 62.109 0)
+      (effects (font (size 1.27 1.27)) (justify left))
+    )

Commit message: WIP
Parts:
- removed J5: Barrel_Jack, symbol Connector:Barrel_Jack
Connections:
- net 12Vin renamed +12V
Other:
- note removed: "External Power"
Changed lines of the file:
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@@
-    (stroke (width 0) (type solid) (color 0 0 0 0))
-  )
-  (wire (pts (xy 41.91 34.29) (xy 44.45 34.29))
-    (stroke (width 0) (type solid) (color 0 0 0 0))
-  )
-  (wire (pts (xy 41.91 39.37) (xy 44.45 39.37))
-    (stroke (width 0) (type solid) (color 0 0 0 0))
-  )
-  (wire (pts (xy 44.45 31.75) (xy 44.45 34.29))
-    (stroke (width 0) (type solid) (color 0 0 0 0))
-  )
-  (wire (pts (xy 44.45 39.37) (xy 44.45 41.91))
     (stroke (width 0) (type solid) (color 0 0 0 0))
   )
@@
     (stroke (width 0) (type solid) (color 0 0 0 0))
   )
+  (wire (pts (xy 101.6 46.99) (xy 101.6 49.53))
+    (stroke (width 0) (type solid) (color 0 0 0 0))
+  )
   (wire (pts (xy 101.6 49.53) (xy 105.41 49.53))
     (stroke (width 0) (type solid) (color 0 0 0 0))
@@
   )
   (text "TODO:\n - Bus power input (From DC to DC converter in battery\n - Bus power delivery"
-    (at 22.86 60.96 0)
+    (at 21.59 111.76 0)
     (effects (font (size 1.27 1.27)) (justify left bottom))
   )
@@
     (effects (font (size 1.27 1.27)) (justify left bottom))
   )
-  (text "External Power" (at 39.37 45.72 180)
-    (effects (font (size 1.27 1.27)) (justify right bottom))
-  )
   (text "Use at least 1% precision resistors" (at 55.88 154.94 0)
     (effects (font (size 1.27 1.27)) (justify left bottom))
@@
     (effects (font (size 1.27 1.27)) (justify right bottom))
   )
-  (hierarchical_label "12Vin" (shape input) (at 101.6 49.53 180)
-    (effects (font (size 1.27 1.27)) (justify right))
-  )
   (hierarchical_label "5Vout" (shape output) (at 196.85 52.07 0)
     (effects (font (size 1.27 1.27)) (justify left))
+  )
+  (symbol (lib_id "power:+12V") (at 101.6 46.99 0) (unit 1)
+    (in_bom yes) (on_board yes)
+    (property "Reference" "#PWR05" (id 0) (at 101.6 50.8 0)
+      (effects (font (size 1.27 1.27)) hide)
+    )
+    (property "Value" "+12V" (id 1) (at 101.9683 42.6656 0))
+    (property "Footprint" "" (id 2) (at 101.6 46.99 0)
+      (effects (font (size 1.27 1.27)) hide)
+    )
+    (property "Datasheet" "" (id 3) (at 101.6 46.99 0)
+      (effects (font (size 1.27 1.27)) hide)
+    )
   )
   (symbol (lib_id "symbols:3.3uH") (at 158.75 52.07 90) (unit 1)
@@
     )
   )
-  (symbol (lib_id "power:GND") (at 44.45 41.91 0) (unit 1)
-    (in_bom yes) (on_board yes)
-    (property "Reference" "#PWR0118" (id 0) (at 44.45 48.26 0)
-      (effects (font (size 1.27 1.27)) hide)
-    )
-    (property "Value" "GND" (id 1) (at 44.5643 46.2344 0))
-    (property "Footprint" "" (id 2) (at 44.45 41.91 0)
-      (effects (font (size 1.27 1.27)) hide)
-    )
-    (property "Datasheet" "" (id 3) (at 44.45 41.91 0)
-      (effects (font (size 1.27 1.27)) hide)
-    )
-  )
   (symbol (lib_id "power:GND") (at 49.53 172.72 0) (unit 1)
     (in_bom yes) (on_board yes)
@@
       (effects (font (size 1.27 1.27)) hide)
     )
-  )
-  (symbol (lib_id "Connector:Barrel_Jack") (at 34.29 36.83 0) (unit 1)
-    (in_bom yes) (on_board yes)
-    (property "Reference" "J5" (id 0) (at 35.687 28.7082 0))
-    (property "Value" "Barrel_Jack" (id 1) (at 35.687 31.0069 0))
-    (property "Footprint" "" (id 2) (at 35.56 37.846 0)
-      (effects (font (size 1.27 1.27)) hide)
-    )
-    (property "Datasheet" "~" (id 3) (at 35.56 37.846 0)
-      (effects (font (size 1.27 1.27)) hide)
-    )

Commit message: footprint assignments
Parts:
- JP4: footprint (none) -> Jumper:SolderJumper-2_P1.3mm_Open_RoundedPad1.0x1.5mm
- U3: footprint (none) -> Package_SO:SOIC-8-1EP_3.9x4.9mm_P1.27mm_EP2.514x3.2mm
Changed lines of the file:
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@@
   (symbol (lib_id "power:+12V") (at 101.6 46.99 0) (unit 1)
     (in_bom yes) (on_board yes)
-    (property "Reference" "#PWR05" (id 0) (at 101.6 50.8 0)
+    (property "Reference" "#PWR0123" (id 0) (at 101.6 50.8 0)
       (effects (font (size 1.27 1.27)) hide)
     )
@@
   (symbol (lib_id "power:GND") (at 49.53 172.72 0) (unit 1)
     (in_bom yes) (on_board yes)
-    (property "Reference" "#PWR0116" (id 0) (at 49.53 179.07 0)
+    (property "Reference" "#PWR0120" (id 0) (at 49.53 179.07 0)
       (effects (font (size 1.27 1.27)) hide)
     )
@@
   (symbol (lib_id "power:GND") (at 114.3 172.72 0) (unit 1)
     (in_bom yes) (on_board yes)
-    (property "Reference" "#PWR0115" (id 0) (at 114.3 179.07 0)
+    (property "Reference" "#PWR0121" (id 0) (at 114.3 179.07 0)
       (effects (font (size 1.27 1.27)) hide)
     )
@@
   (symbol (lib_id "power:GND") (at 139.7 71.12 0) (unit 1)
     (in_bom yes) (on_board yes)
-    (property "Reference" "#PWR0119" (id 0) (at 139.7 77.47 0)
+    (property "Reference" "#PWR0122" (id 0) (at 139.7 77.47 0)
       (effects (font (size 1.27 1.27)) hide)
     )
@@
       (effects (font (size 1.27 1.27)) (justify right))
     )
-    (property "Footprint" "" (id 2) (at 123.19 160.02 0)
+    (property "Footprint" "Jumper:SolderJumper-2_P1.3mm_Open_RoundedPad1.0x1.5mm" (id 2) (at 123.19 160.02 0)
       (effects (font (size 1.27 1.27)) hide)
     )
@@
     (property "Reference" "U3" (id 0) (at 132.715 42.9065 0))
     (property "Value" "AP64501" (id 1) (at 132.715 45.2052 0))
-    (property "Footprint" "" (id 2) (at 121.92 52.07 0)
-      (effects (font (size 1.27 1.27)) hide)
-    )
-    (property "Datasheet" "" (id 3) (at 121.92 52.07 0)
-      (effects (font (size 1.27 1.27)) hide)
-    )
+    (property "Footprint" "Package_SO:SOIC-8-1EP_3.9x4.9mm_P1.27mm_EP2.514x3.2mm" (id 2) (at 121.92 52.07 0)
+      (effects (font (size 1.27 1.27)) hide)
+    )
+    (property "Datasheet" "https://www.diodes.com/assets/Datasheets/AP64501.pdf" (id 3) (at 121.92 52.07 0)
+      (effects (font (size 1.27 1.27)) hide)
+    )
