File: power.kicad_sch (KiCad schematic)
At the start: 24 parts, among them J1 Barrel_Jack, U1 AP64501, U9 TPS79933

Commit message: WIP
Parts:
- added D?: LED_Green, LED_SMD:LED_0805_2012Metric_Pad1.15x1.40mm_HandSolder, symbol ecafe-racer:LED_Green
- added R?: R, Resistor_SMD:R_0805_2012Metric, symbol Device:R
Connections:
- net GND: now also R?.2
- net PWR_IN: now also D?.2
- new net: D?.1, R?.1
Other:
- note added: "12V Supply Power Indicator"
Changed lines of the file:
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@@
+    (stroke (width 0) (type solid) (color 0 0 0 0))
+  )
+  (wire (pts (xy 113.03 165.1) (xy 113.03 176.53))
     (stroke (width 0) (type solid) (color 0 0 0 0))
   )
@@
     (effects (font (size 1.27 1.27)) (justify left bottom))
   )
+  (text "12V Supply Power Indicator" (at 124.46 193.04 90)
+    (effects (font (size 1.27 1.27)) (justify left bottom))
+  )
   (text "Feedback Circuit\n\nVout is determined by this feedback\ndivider circuit with the equation:\nR_{high} = R_{low} * (V_{out} / 0.8V - 1)\n\n*C4 is optional for improving transient response\n*Use at least 1% precision resistors"
     (at 180.34 165.735 0)
@@
     (effects (font (size 1.27 1.27)) (justify left bottom))
   )
+  (label "PWR_IN" (at 113.03 165.1 270)
+    (effects (font (size 1.27 1.27)) (justify right bottom))
+  )
   (label "feedback" (at 140.97 43.815 180)
     (effects (font (size 1.27 1.27)) (justify right bottom))
@@
     )
     (property "Datasheet" "" (id 3) (at 109.22 111.76 0)
+      (effects (font (size 1.27 1.27)) hide)
+    )
+    (pin "1")
+  )
+  (symbol (lib_id "power:GND") (at 113.03 191.77 0) (unit 1)
+    (in_bom yes) (on_board yes) (fields_autoplaced)
+    (property "Reference" "#PWR?" (id 0) (at 113.03 198.12 0)
+      (effects (font (size 1.27 1.27)) hide)
+    )
+    (property "Value" "GND" (id 1) (at 113.03 196.85 0))
+    (property "Footprint" "" (id 2) (at 113.03 191.77 0)
+      (effects (font (size 1.27 1.27)) hide)
+    )
+    (property "Datasheet" "" (id 3) (at 113.03 191.77 0)
       (effects (font (size 1.27 1.27)) hide)
     )
@@
     (pin "2")
   )
+  (symbol (lib_id "Device:R") (at 113.03 187.96 0) (unit 1)
+    (in_bom yes) (on_board yes) (fields_autoplaced)
+    (property "Reference" "R?" (id 0) (at 115.57 186.6899 0)
+      (effects (font (size 1.27 1.27)) (justify left))
+    )
+    (property "Value" "R" (id 1) (at 115.57 189.2299 0)
+      (effects (font (size 1.27 1.27)) (justify left))
+    )
+    (property "Footprint" "Resistor_SMD:R_0805_2012Metric" (id 2) (at 111.252 187.96 90)
+      (effects (font (size 1.27 1.27)) hide)
+    )
+    (property "Datasheet" "~" (id 3) (at 113.03 187.96 0)
+      (effects (font (size 1.27 1.27)) hide)
+    )
+    (pin "1")
+    (pin "2")
+  )
   (symbol (lib_id "Device:R") (at 194.31 125.095 0) (unit 1)
     (in_bom yes) (on_board yes)
@@
       (effects (font (size 1.27 1.27)) hide)
     )
+    (pin "1")
+    (pin "2")
+  )
+  (symbol (lib_id "ecafe-racer:LED_Green") (at 113.03 180.34 90) (unit 1)
+    (in_bom yes) (on_board yes) (fields_autoplaced)
+    (property "Reference" "D?" (id 0) (at 116.84 179.2604 90)
+      (effects (font (size 1.27 1.27)) (justify right))
+    )
+    (property "Value" "LED_Green" (id 1) (at 116.84 181.8004 90)
+      (effects (font (size 1.27 1.27)) (justify right) hide)
+    )
+    (property "Footprint" "LED_SMD:LED_0805_2012Metric_Pad1.15x1.40mm_HandSolder" (id 2) (at 101.6 171.45 0)
+      (effects (font (size 1.27 1.27)) hide)
+    )
+    (property "Datasheet" "https://vcclite.com/wp-content/uploads/wpallimport/files/files/CMD1721Seriesver3.pdf" (id 3) (at 109.22 176.53 0)
+      (effects (font (size 1.27 1.27)) hide)
+    )
+    (property "Vendor" "Digikey" (id 4) (at 93.98 198.12 0)
+      (effects (font (size 1.27 1.27)) hide)
+    )
+    (property "Vendor Part" "L62405CT-ND" (id 5) (at 96.52 194.31 0)
+      (effects (font (size 1.27 1.27)) hide)
+    )
+    (property "Manufacturer" "Visual Communications Company - VCC" (id 6) (at 104.14 181.61 0)
+      (effects (font (size 1.27 1.27)) hide)
+    )
+    (property "Manufacturer Part" "CMD17-21VGC/TR8" (id 7) (at 99.06 191.77 0)
+      (effects (font (size 1.27 1.27)) hide)
+    )

Commit message: WIP
Parts:
- gave numbers to parts that had none: 2
Changed lines of the file:
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@@
   (symbol (lib_id "power:GND") (at 113.03 191.77 0) (unit 1)
     (in_bom yes) (on_board yes) (fields_autoplaced)
-    (property "Reference" "#PWR?" (id 0) (at 113.03 198.12 0)
+    (property "Reference" "#PWR0147" (id 0) (at 113.03 198.12 0)
       (effects (font (size 1.27 1.27)) hide)
     )
@@
   (symbol (lib_id "Device:R") (at 113.03 187.96 0) (unit 1)
     (in_bom yes) (on_board yes) (fields_autoplaced)
-    (property "Reference" "R?" (id 0) (at 115.57 186.6899 0)
+    (property "Reference" "R31" (id 0) (at 115.57 186.6899 0)
       (effects (font (size 1.27 1.27)) (justify left))
     )
@@
   (symbol (lib_id "ecafe-racer:LED_Green") (at 113.03 180.34 90) (unit 1)
     (in_bom yes) (on_board yes) (fields_autoplaced)
-    (property "Reference" "D?" (id 0) (at 116.84 179.2604 90)
+    (property "Reference" "D19" (id 0) (at 116.84 179.2604 90)
       (effects (font (size 1.27 1.27)) (justify right))
     )
