File: real_time_clock.kicad_sch (KiCad schematic)
At the start: 4 parts

Commit message: Added buses and USB ports to schematic
Parts:
- gave numbers to parts that had none: 4
Other:
- company: (none) -> eCafe Racer
- title: (none) -> Dennis
Changed lines of the file:
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@@
 (kicad_sch (version 20201015) (generator eeschema)
-  (paper "A4")
+  (paper "A")
+  (title_block
+    (title "Dennis")
+    (date "2020-12-31")
+    (rev "0.1.1")
+    (company "eCafe Racer")
+  )
   (no_connect (at 97.79 106.68))
   (no_connect (at 116.84 104.14))
@@
   (symbol (lib_id "power:+3.3V") (at 62.23 104.14 0) (unit 1)
     (in_bom yes) (on_board yes)
-    (property "Reference" "#PWR?" (id 0) (at 62.23 107.95 0)
+    (property "Reference" "#PWR031" (id 0) (at 62.23 107.95 0)
       (effects (font (size 1.27 1.27)) hide)
     )
@@
   (symbol (lib_id "power:GND") (at 62.23 124.46 0) (unit 1)
     (in_bom yes) (on_board yes)
-    (property "Reference" "#PWR?" (id 0) (at 62.23 130.81 0)
+    (property "Reference" "#PWR032" (id 0) (at 62.23 130.81 0)
       (effects (font (size 1.27 1.27)) hide)
     )
@@
   (symbol (lib_id "power:GND") (at 96.52 110.49 0) (unit 1)
     (in_bom yes) (on_board yes)
-    (property "Reference" "#PWR?" (id 0) (at 96.52 116.84 0)
+    (property "Reference" "#PWR033" (id 0) (at 96.52 116.84 0)
       (effects (font (size 1.27 1.27)) hide)
     )
@@
   (symbol (lib_id "Device:Battery_Cell") (at 62.23 121.92 0) (unit 1)
     (in_bom yes) (on_board yes)
-    (property "Reference" "BT?" (id 0) (at 65.1511 119.5006 0)
+    (property "Reference" "BT1" (id 0) (at 65.1511 119.5006 0)
       (effects (font (size 1.27 1.27)) (justify left))
     )
@@
   (symbol (lib_id "Device:Crystal") (at 102.87 129.54 90) (unit 1)
     (in_bom yes) (on_board yes)
-    (property "Reference" "Y?" (id 0) (at 93.4975 128.3906 90)
+    (property "Reference" "Y2" (id 0) (at 93.4975 128.3906 90)
       (effects (font (size 1.27 1.27)) (justify right))
     )
@@
   (symbol (lib_id "symbols:BAT54C-7-F") (at 62.23 110.49 0) (unit 1)
     (in_bom yes) (on_board yes)
-    (property "Reference" "D?" (id 0) (at 60.198 109.3406 0)
+    (property "Reference" "D1" (id 0) (at 60.198 109.3406 0)
       (effects (font (size 1.27 1.27)) (justify right))
     )
@@
   (symbol (lib_id "symbols:PCF85063A") (at 107.95 105.41 0) (unit 1)
     (in_bom yes) (on_board yes)
-    (property "Reference" "U?" (id 0) (at 107.315 94.9765 0))
+    (property "Reference" "U6" (id 0) (at 107.315 94.9765 0))
     (property "Value" "PCF85063A" (id 1) (at 107.315 97.2752 0))
     (property "Footprint" "" (id 2) (at 101.6 102.87 0)

Commit message: footprints
Parts:
- renumbered D1 to D2, U6 to U7
Changed lines of the file:
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@@
   (symbol (lib_id "power:+3.3V") (at 62.23 104.14 0) (unit 1)
     (in_bom yes) (on_board yes)
-    (property "Reference" "#PWR031" (id 0) (at 62.23 107.95 0)
+    (property "Reference" "#PWR0150" (id 0) (at 62.23 107.95 0)
       (effects (font (size 1.27 1.27)) hide)
     )
@@
   (symbol (lib_id "power:GND") (at 62.23 124.46 0) (unit 1)
     (in_bom yes) (on_board yes)
-    (property "Reference" "#PWR032" (id 0) (at 62.23 130.81 0)
+    (property "Reference" "#PWR0151" (id 0) (at 62.23 130.81 0)
       (effects (font (size 1.27 1.27)) hide)
     )
@@
   (symbol (lib_id "power:GND") (at 96.52 110.49 0) (unit 1)
     (in_bom yes) (on_board yes)
-    (property "Reference" "#PWR033" (id 0) (at 96.52 116.84 0)
+    (property "Reference" "#PWR0152" (id 0) (at 96.52 116.84 0)
       (effects (font (size 1.27 1.27)) hide)
     )
@@
   (symbol (lib_id "symbols:BAT54C-7-F") (at 62.23 110.49 0) (unit 1)
     (in_bom yes) (on_board yes)
-    (property "Reference" "D1" (id 0) (at 60.198 109.3406 0)
+    (property "Reference" "D2" (id 0) (at 60.198 109.3406 0)
       (effects (font (size 1.27 1.27)) (justify right))
     )
@@
   (symbol (lib_id "symbols:PCF85063A") (at 107.95 105.41 0) (unit 1)
     (in_bom yes) (on_board yes)
-    (property "Reference" "U6" (id 0) (at 107.315 94.9765 0))
+    (property "Reference" "U7" (id 0) (at 107.315 94.9765 0))
     (property "Value" "PCF85063A" (id 1) (at 107.315 97.2752 0))
     (property "Footprint" "" (id 2) (at 101.6 102.87 0)

Commit message: footprint assignments
Parts:
- removed BT1: Battery_Cell, symbol Device:Battery_Cell
- added BT1: Battery_Cell, Battery:BatteryHolder_Keystone_3001_1x12mm, symbol symbols:Battery_Cell
- U7: footprint (none) -> Package_SO:SOIC-8_3.9x4.9mm_P1.27mm
- renumbered D2 to D3
Connections:
- net GND: now also BT1.2 (-)
- net at D3.2 (Anode_{2}): now also BT1.1 (+)
Changed lines of the file:
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@@
   (symbol (lib_id "power:+3.3V") (at 62.23 104.14 0) (unit 1)
     (in_bom yes) (on_board yes)
-    (property "Reference" "#PWR0150" (id 0) (at 62.23 107.95 0)
+    (property "Reference" "#PWR0155" (id 0) (at 62.23 107.95 0)
       (effects (font (size 1.27 1.27)) hide)
     )
@@
   (symbol (lib_id "power:GND") (at 62.23 124.46 0) (unit 1)
     (in_bom yes) (on_board yes)
-    (property "Reference" "#PWR0151" (id 0) (at 62.23 130.81 0)
+    (property "Reference" "#PWR0154" (id 0) (at 62.23 130.81 0)
       (effects (font (size 1.27 1.27)) hide)
     )
@@
   (symbol (lib_id "power:GND") (at 96.52 110.49 0) (unit 1)
     (in_bom yes) (on_board yes)
-    (property "Reference" "#PWR0152" (id 0) (at 96.52 116.84 0)
+    (property "Reference" "#PWR0156" (id 0) (at 96.52 116.84 0)
       (effects (font (size 1.27 1.27)) hide)
     )
@@
     )
   )
-  (symbol (lib_id "Device:Battery_Cell") (at 62.23 121.92 0) (unit 1)
+  (symbol (lib_id "symbols:Battery_Cell") (at 62.23 121.92 0) (unit 1)
     (in_bom yes) (on_board yes)
-    (property "Reference" "BT1" (id 0) (at 65.1511 119.5006 0)
+    (property "Reference" "BT1" (id 0) (at 65.151 119.501 0)
       (effects (font (size 1.27 1.27)) (justify left))
     )
     (property "Value" "Battery_Cell" (id 1) (at 65.1511 121.7993 0)
-      (effects (font (size 1.27 1.27)) (justify left) hide)
+      (effects (font (size 1.27 1.27)) (justify left))
     )
-    (property "Footprint" "" (id 2) (at 62.23 120.396 90)
+    (property "Footprint" "Battery:BatteryHolder_Keystone_3001_1x12mm" (id 2) (at 62.23 120.396 90)
       (effects (font (size 1.27 1.27)) hide)
     )
-    (property "Datasheet" "~" (id 3) (at 62.23 120.396 90)
+    (property "Datasheet" "https://www.keyelco.com/userAssets/file/M65p9.pdf" (id 3) (at 62.23 120.396 90)
       (effects (font (size 1.27 1.27)) hide)
     )
-    (property "Voltage" "3.3V" (id 4) (at 67.31 121.92 0))
+    (property "Drawing" "www.keyelco.com/product-pdf.cfm?p=778" (id 4) (at 62.23 121.92 0)
+      (effects (font (size 1.27 1.27)) hide)
+    )
+    (property "Vendor" "Digikey" (id 5) (at 62.23 121.92 0)
+      (effects (font (size 1.27 1.27)) hide)
+    )
+    (property "Vendor Part" "36-3001-ND" (id 6) (at 62.23 121.92 0)
+      (effects (font (size 1.27 1.27)) hide)
+    )
+    (property "Manufacturer" "Keystone Electronics" (id 7) (at 62.23 121.92 0)
+      (effects (font (size 1.27 1.27)) hide)
+    )
+    (property "Manufacturer Part" "3001" (id 8) (at 62.23 121.92 0)
+      (effects (font (size 1.27 1.27)) hide)
+    )
   )
   (symbol (lib_id "Device:Crystal") (at 102.87 129.54 90) (unit 1)
@@
   (symbol (lib_id "symbols:BAT54C-7-F") (at 62.23 110.49 0) (unit 1)
     (in_bom yes) (on_board yes)
-    (property "Reference" "D2" (id 0) (at 60.198 109.3406 0)
+    (property "Reference" "D3" (id 0) (at 60.198 109.3406 0)
       (effects (font (size 1.27 1.27)) (justify right))
     )
@@
     (property "Reference" "U7" (id 0) (at 107.315 94.9765 0))
     (property "Value" "PCF85063A" (id 1) (at 107.315 97.2752 0))
-    (property "Footprint" "" (id 2) (at 101.6 102.87 0)
+    (property "Footprint" "Package_SO:SOIC-8_3.9x4.9mm_P1.27mm" (id 2) (at 101.6 102.87 0)
       (effects (font (size 1.27 1.27)) hide)
     )

Commit message: WIP 5 FEB 2021
Parts:
- U7: footprint Package_SO:SOIC-8_3.9x4.9mm_P1.27mm -> (none)
Changed lines of the file:
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@@
     (property "Reference" "U7" (id 0) (at 107.315 94.9765 0))
     (property "Value" "PCF85063A" (id 1) (at 107.315 97.2752 0))
-    (property "Footprint" "Package_SO:SOIC-8_3.9x4.9mm_P1.27mm" (id 2) (at 101.6 102.87 0)
+    (property "Footprint" "" (id 2) (at 101.6 102.87 0)
       (effects (font (size 1.27 1.27)) hide)
     )
