File: compute_module_B.kicad_sch (KiCad schematic)
At the start: 3 parts, among them J10 HDMI_A_1.4, U8 TUSB2046IBVF

Commit message: more layout: power supply and gpio
Parts:
- renumbered J10 to J14, U8 to U2
Changed lines of the file:
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@@
   (junction (at 232.41 88.9) (diameter 0.9144) (color 0 0 0 0))
   (junction (at 234.95 88.9) (diameter 0.9144) (color 0 0 0 0))
+  (no_connect (at 53.34 41.91))
+  (no_connect (at 53.34 105.41))
+  (no_connect (at 53.34 72.39))
+  (no_connect (at 114.3 90.17))
+  (no_connect (at 53.34 92.71))
+  (no_connect (at 114.3 82.55))
+  (no_connect (at 53.34 59.69))
+  (no_connect (at 53.34 49.53))
+  (no_connect (at 53.34 90.17))
+  (no_connect (at 53.34 120.65))
+  (no_connect (at 114.3 52.07))
+  (no_connect (at 114.3 105.41))
+  (no_connect (at 53.34 133.35))
+  (no_connect (at 53.34 143.51))
+  (no_connect (at 114.3 72.39))
+  (no_connect (at 114.3 34.29))
+  (no_connect (at 53.34 118.11))
+  (no_connect (at 53.34 110.49))
+  (no_connect (at 53.34 52.07))
+  (no_connect (at 53.34 87.63))
+  (no_connect (at 114.3 31.75))
+  (no_connect (at 53.34 80.01))
+  (no_connect (at 114.3 49.53))
+  (no_connect (at 114.3 57.15))
+  (no_connect (at 53.34 140.97))
+  (no_connect (at 114.3 97.79))
+  (no_connect (at 114.3 41.91))
+  (no_connect (at 53.34 113.03))
+  (no_connect (at 114.3 74.93))
+  (no_connect (at 53.34 148.59))
+  (no_connect (at 114.3 36.83))
+  (no_connect (at 53.34 135.89))
+  (no_connect (at 114.3 95.25))
+  (no_connect (at 114.3 87.63))
+  (no_connect (at 114.3 67.31))
+  (no_connect (at 53.34 82.55))
+  (no_connect (at 53.34 44.45))
+  (no_connect (at 53.34 102.87))
   (no_connect (at 114.3 59.69))
-  (no_connect (at 53.34 92.71))
-  (no_connect (at 53.34 110.49))
-  (no_connect (at 53.34 143.51))
-  (no_connect (at 114.3 67.31))
+  (no_connect (at 53.34 67.31))
+  (no_connect (at 53.34 57.15))
+  (no_connect (at 53.34 74.93))
+  (no_connect (at 114.3 113.03))
+  (no_connect (at 114.3 64.77))
+  (no_connect (at 114.3 80.01))
   (no_connect (at 114.3 102.87))
-  (no_connect (at 53.34 118.11))
+  (no_connect (at 53.34 85.09))
+  (no_connect (at 114.3 44.45))
+  (no_connect (at 53.34 151.13))
+  (no_connect (at 53.34 128.27))
   (no_connect (at 53.34 125.73))
-  (no_connect (at 114.3 57.15))
-  (no_connect (at 53.34 87.63))
-  (no_connect (at 114.3 41.91))
-  (no_connect (at 53.34 135.89))
-  (no_connect (at 53.34 140.97))
-  (no_connect (at 114.3 105.41))
-  (no_connect (at 114.3 87.63))
-  (no_connect (at 53.34 133.35))
-  (no_connect (at 53.34 49.53))
-  (no_connect (at 114.3 44.45))
+  (no_connect (at 53.34 64.77))
   (no_connect (at 114.3 110.49))
-  (no_connect (at 114.3 95.25))
-  (no_connect (at 53.34 82.55))
-  (no_connect (at 53.34 151.13))
-  (no_connect (at 53.34 120.65))
-  (no_connect (at 114.3 74.93))
-  (no_connect (at 114.3 113.03))
-  (no_connect (at 114.3 52.07))
-  (no_connect (at 53.34 41.91))
-  (no_connect (at 53.34 80.01))
-  (no_connect (at 53.34 57.15))
-  (no_connect (at 114.3 64.77))
-  (no_connect (at 114.3 31.75))
-  (no_connect (at 53.34 74.93))
-  (no_connect (at 53.34 52.07))
-  (no_connect (at 114.3 82.55))
-  (no_connect (at 53.34 85.09))
-  (no_connect (at 53.34 67.31))
-  (no_connect (at 53.34 59.69))
-  (no_connect (at 53.34 64.77))
-  (no_connect (at 53.34 90.17))
-  (no_connect (at 53.34 102.87))
-  (no_connect (at 114.3 49.53))
-  (no_connect (at 53.34 148.59))
-  (no_connect (at 114.3 97.79))
-  (no_connect (at 114.3 80.01))
-  (no_connect (at 53.34 44.45))
-  (no_connect (at 114.3 34.29))
-  (no_connect (at 114.3 90.17))
-  (no_connect (at 114.3 72.39))
-  (no_connect (at 114.3 36.83))
-  (no_connect (at 53.34 72.39))
-  (no_connect (at 53.34 105.41))
-  (no_connect (at 53.34 128.27))
-  (no_connect (at 53.34 113.03))
   (bus_entry (at 31.75 97.79) (size 2.54 -2.54)
     (stroke (width 0.1524) (type solid) (color 0 0 0 0))
@@
   (symbol (lib_id "power:+5V") (at 227.33 30.48 0) (unit 1)
     (in_bom yes) (on_board yes)
-    (property "Reference" "#PWR0159" (id 0) (at 227.33 34.29 0)
+    (property "Reference" "#PWR0136" (id 0) (at 227.33 34.29 0)
       (effects (font (size 1.27 1.27)) hide)
     )
@@
   (symbol (lib_id "power:GND") (at 50.8 160.02 0) (unit 1)
     (in_bom yes) (on_board yes)
-    (property "Reference" "#PWR0157" (id 0) (at 50.8 166.37 0)
+    (property "Reference" "#PWR0133" (id 0) (at 50.8 166.37 0)
       (effects (font (size 1.27 1.27)) hide)
     )
@@
   (symbol (lib_id "power:GND") (at 116.84 160.02 0) (unit 1)
     (in_bom yes) (on_board yes)
-    (property "Reference" "#PWR0158" (id 0) (at 116.84 166.37 0)
+    (property "Reference" "#PWR0134" (id 0) (at 116.84 166.37 0)
       (effects (font (size 1.27 1.27)) hide)
     )
@@
   (symbol (lib_id "power:GND") (at 234.95 91.44 0) (unit 1)
     (in_bom yes) (on_board yes)
-    (property "Reference" "#PWR0160" (id 0) (at 234.95 97.79 0)
+    (property "Reference" "#PWR0135" (id 0) (at 234.95 97.79 0)
       (effects (font (size 1.27 1.27)) hide)
     )
@@
   (symbol (lib_id "symbols:HDMI_A_1.4") (at 227.33 58.42 0) (unit 1)
     (in_bom yes) (on_board yes)
-    (property "Reference" "J10" (id 0) (at 238.2521 57.2706 0)
+    (property "Reference" "J14" (id 0) (at 238.2521 57.2706 0)
       (effects (font (size 1.27 1.27)) (justify left))
     )
@@
   (symbol (lib_id "symbols:TUSB2046IBVF") (at 229.87 133.35 0) (mirror y) (unit 1)
     (in_bom yes) (on_board yes)
-    (property "Reference" "U8" (id 0) (at 229.235 106.4065 0))
+    (property "Reference" "U2" (id 0) (at 229.235 106.4065 0))
     (property "Value" "TUSB2046IBVF" (id 1) (at 229.235 108.7052 0))
     (property "Footprint" "Package_QFP:LQFP-32_7x7mm_P0.8mm" (id 2) (at 224.79 107.95 0)

Commit message: Routing for HDMI, Ethernet, SD Card, CAN
Parts:
- added C21: 0.1uF, Capacitor_SMD:C_0805_2012Metric, symbol Device:C
Connections:
- net GND: now also C21.2
- net +3V3: now reaches U2.26 (~EXTMEM)
- net +3V3: now also U2.8 (BUSPWR), C21.1
- no-connect marks 53 -> 54
Other:
- note removed: "TODO: make of find footprint"
Changed lines of the file:
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@@
   (junction (at 116.84 146.05) (diameter 0.9144) (color 0 0 0 0))
   (junction (at 116.84 153.67) (diameter 0.9144) (color 0 0 0 0))
+  (junction (at 199.39 124.46) (diameter 0.9144) (color 0 0 0 0))
   (junction (at 224.79 88.9) (diameter 0.9144) (color 0 0 0 0))
   (junction (at 227.33 88.9) (diameter 0.9144) (color 0 0 0 0))
@@
   (junction (at 232.41 88.9) (diameter 0.9144) (color 0 0 0 0))
   (junction (at 234.95 88.9) (diameter 0.9144) (color 0 0 0 0))
+  (no_connect (at 114.3 90.17))
+  (no_connect (at 114.3 113.03))
+  (no_connect (at 53.34 52.07))
+  (no_connect (at 53.34 125.73))
+  (no_connect (at 53.34 140.97))
+  (no_connect (at 53.34 102.87))
+  (no_connect (at 53.34 74.93))
+  (no_connect (at 114.3 72.39))
+  (no_connect (at 114.3 52.07))
+  (no_connect (at 53.34 64.77))
+  (no_connect (at 114.3 31.75))
+  (no_connect (at 53.34 92.71))
+  (no_connect (at 114.3 57.15))
+  (no_connect (at 114.3 34.29))
+  (no_connect (at 53.34 151.13))
+  (no_connect (at 53.34 143.51))
+  (no_connect (at 53.34 82.55))
+  (no_connect (at 114.3 82.55))
   (no_connect (at 53.34 41.91))
-  (no_connect (at 53.34 105.41))
-  (no_connect (at 53.34 72.39))
-  (no_connect (at 114.3 90.17))
-  (no_connect (at 53.34 92.71))
-  (no_connect (at 114.3 82.55))
-  (no_connect (at 53.34 59.69))
-  (no_connect (at 53.34 49.53))
-  (no_connect (at 53.34 90.17))
+  (no_connect (at 114.3 41.91))
+  (no_connect (at 114.3 105.41))
+  (no_connect (at 53.34 113.03))
+  (no_connect (at 53.34 110.49))
+  (no_connect (at 53.34 128.27))
+  (no_connect (at 114.3 80.01))
+  (no_connect (at 213.36 127))
+  (no_connect (at 114.3 44.45))
   (no_connect (at 53.34 120.65))
-  (no_connect (at 114.3 52.07))
-  (no_connect (at 114.3 105.41))
-  (no_connect (at 53.34 133.35))
-  (no_connect (at 53.34 143.51))
-  (no_connect (at 114.3 72.39))
-  (no_connect (at 114.3 34.29))
-  (no_connect (at 53.34 118.11))
-  (no_connect (at 53.34 110.49))
-  (no_connect (at 53.34 52.07))
-  (no_connect (at 53.34 87.63))
-  (no_connect (at 114.3 31.75))
+  (no_connect (at 53.34 135.89))
+  (no_connect (at 53.34 57.15))
+  (no_connect (at 114.3 95.25))
+  (no_connect (at 114.3 74.93))
   (no_connect (at 53.34 80.01))
-  (no_connect (at 114.3 49.53))
-  (no_connect (at 114.3 57.15))
-  (no_connect (at 53.34 140.97))
-  (no_connect (at 114.3 97.79))
-  (no_connect (at 114.3 41.91))
-  (no_connect (at 53.34 113.03))
-  (no_connect (at 114.3 74.93))
-  (no_connect (at 53.34 148.59))
-  (no_connect (at 114.3 36.83))
-  (no_connect (at 53.34 135.89))
-  (no_connect (at 114.3 95.25))
-  (no_connect (at 114.3 87.63))
-  (no_connect (at 114.3 67.31))
-  (no_connect (at 53.34 82.55))
-  (no_connect (at 53.34 44.45))
-  (no_connect (at 53.34 102.87))
   (no_connect (at 114.3 59.69))
   (no_connect (at 53.34 67.31))
-  (no_connect (at 53.34 57.15))
-  (no_connect (at 53.34 74.93))
-  (no_connect (at 114.3 113.03))
+  (no_connect (at 114.3 49.53))
+  (no_connect (at 114.3 87.63))
+  (no_connect (at 53.34 133.35))
+  (no_connect (at 114.3 36.83))
+  (no_connect (at 114.3 67.31))
+  (no_connect (at 53.34 148.59))
+  (no_connect (at 53.34 118.11))
+  (no_connect (at 53.34 105.41))
+  (no_connect (at 53.34 49.53))
+  (no_connect (at 114.3 110.49))
+  (no_connect (at 114.3 102.87))
+  (no_connect (at 53.34 90.17))
   (no_connect (at 114.3 64.77))
-  (no_connect (at 114.3 80.01))
-  (no_connect (at 114.3 102.87))
+  (no_connect (at 53.34 59.69))
   (no_connect (at 53.34 85.09))
-  (no_connect (at 114.3 44.45))
-  (no_connect (at 53.34 151.13))
-  (no_connect (at 53.34 128.27))
-  (no_connect (at 53.34 125.73))
-  (no_connect (at 53.34 64.77))
-  (no_connect (at 114.3 110.49))
+  (no_connect (at 53.34 44.45))
+  (no_connect (at 53.34 72.39))
+  (no_connect (at 114.3 97.79))
+  (no_connect (at 53.34 87.63))
   (bus_entry (at 31.75 97.79) (size 2.54 -2.54)
     (stroke (width 0.1524) (type solid) (color 0 0 0 0))
@@
     (stroke (width 0) (type solid) (color 0 0 0 0))
   )
+  (wire (pts (xy 199.39 121.92) (xy 199.39 124.46))
+    (stroke (width 0) (type solid) (color 0 0 0 0))
+  )
+  (wire (pts (xy 199.39 124.46) (xy 213.36 124.46))
+    (stroke (width 0) (type solid) (color 0 0 0 0))
+  )
+  (wire (pts (xy 199.39 132.08) (xy 199.39 124.46))
+    (stroke (width 0) (type solid) (color 0 0 0 0))
+  )
   (wire (pts (xy 203.2 60.96) (xy 217.17 60.96))
     (stroke (width 0) (type solid) (color 0 0 0 0))
@@
   )
   (wire (pts (xy 204.47 115.57) (xy 213.36 115.57))
+    (stroke (width 0) (type solid) (color 0 0 0 0))
+  )
+  (wire (pts (xy 213.36 132.08) (xy 199.39 132.08))
     (stroke (width 0) (type solid) (color 0 0 0 0))
   )
@@
     (effects (font (size 1.27 1.27)) (justify right bottom))
   )
-  (text "TODO: make of find footprint" (at 214.63 20.32 0)
-    (effects (font (size 1.27 1.27)) (justify left bottom))
-  )
   (label "USB_{D-}" (at 41.91 34.29 0)
     (effects (font (size 1.27 1.27)) (justify left bottom))
@@
   (hierarchical_label "D_{4}-" (shape bidirectional) (at 250.19 134.62 0)
     (effects (font (size 1.27 1.27)) (justify left))
+  )
+  (symbol (lib_id "power:+3.3V") (at 180.34 116.84 0) (unit 1)
+    (in_bom yes) (on_board yes)
+    (property "Reference" "#PWR0171" (id 0) (at 180.34 120.65 0)
+      (effects (font (size 1.27 1.27)) hide)
+    )
+    (property "Value" "+3.3V" (id 1) (at 180.7083 112.5156 0))
+    (property "Footprint" "" (id 2) (at 180.34 116.84 0)
+      (effects (font (size 1.27 1.27)) hide)
+    )
+    (property "Datasheet" "" (id 3) (at 180.34 116.84 0)
+      (effects (font (size 1.27 1.27)) hide)
+    )
+  )
+  (symbol (lib_id "power:+3.3V") (at 199.39 121.92 0) (unit 1)
+    (in_bom yes) (on_board yes)
+    (property "Reference" "#PWR0170" (id 0) (at 199.39 125.73 0)
+      (effects (font (size 1.27 1.27)) hide)
+    )
+    (property "Value" "+3.3V" (id 1) (at 199.7583 117.5956 0))
+    (property "Footprint" "" (id 2) (at 199.39 121.92 0)
+      (effects (font (size 1.27 1.27)) hide)
+    )
+    (property "Datasheet" "" (id 3) (at 199.39 121.92 0)
+      (effects (font (size 1.27 1.27)) hide)
+    )
   )
   (symbol (lib_id "power:+5V") (at 227.33 30.48 0) (unit 1)
@@
     )
   )
+  (symbol (lib_id "power:GND") (at 180.34 124.46 0) (unit 1)
+    (in_bom yes) (on_board yes)
+    (property "Reference" "#PWR0172" (id 0) (at 180.34 130.81 0)
+      (effects (font (size 1.27 1.27)) hide)
+    )
+    (property "Value" "GND" (id 1) (at 180.4543 128.7844 0))
+    (property "Footprint" "" (id 2) (at 180.34 124.46 0)
+      (effects (font (size 1.27 1.27)) hide)
+    )
+    (property "Datasheet" "" (id 3) (at 180.34 124.46 0)
+      (effects (font (size 1.27 1.27)) hide)
+    )
+  )
   (symbol (lib_id "power:GND") (at 234.95 91.44 0) (unit 1)
     (in_bom yes) (on_board yes)
@@
       (effects (font (size 1.27 1.27)) hide)
     )
+  )
+  (symbol (lib_id "Device:C") (at 180.34 120.65 0) (unit 1)
+    (in_bom yes) (on_board yes)
+    (property "Reference" "C21" (id 0) (at 183.2611 119.5006 0)
+      (effects (font (size 1.27 1.27)) (justify left))
+    )
+    (property "Value" "0.1uF" (id 1) (at 183.261 121.799 0)
+      (effects (font (size 1.27 1.27)) (justify left))
+    )
+    (property "Footprint" "Capacitor_SMD:C_0805_2012Metric" (id 2) (at 181.3052 124.46 0)
+      (effects (font (size 1.27 1.27)) hide)
+    )
+    (property "Datasheet" "~" (id 3) (at 180.34 120.65 0)
+      (effects (font (size 1.27 1.27)) hide)
+    )

Commit message: Finished trace routing
Parts:
- added C4, C5, C6, C8: C, Capacitor_SMD:C_0805_2012Metric, symbol Device:C
- added JP1: SolderJumper_3_Open, Jumper:SolderJumper-3_P1.3mm_Open_RoundedPad1.0x1.5mm_NumberLabels, symbol Jumper:SolderJumper_3_Open
- added R11, R12, R13, R14, R17: R, Resistor_SMD:R_0805_2012Metric, symbol Device:R
- added TP5, TP6, TP7: TestPoint, TestPoint:TestPoint_Pad_D1.5mm, symbol Connector:TestPoint
- added U3: TPS2044BD, Package_SO:SOIC-16_3.9x9.9mm_P1.27mm, symbol symbols:TPS2044BD
- added Y1: HC49USM-FF3F18-6.000MHZ, Crystal:Crystal_SMD_HC49-SD, symbol symbols:HC49USM-FF3F18-6.000MHZ
- C7: renamed from C21; value 0.1uF -> C
Connections:
- net +3V3: now also U2.25 (V_{CC}), U2.3 (V_{CC}), JP1.3 (B), R11.1, R12.1, R13.1, R14.1, R17.1
- net +5V: now also C8.1, U3.2 (IN1), U3.6 (IN2)
- net D_{1}+: now also U2.16 (D_{2}+); no longer U2.12 (D_{1}+)
- net D_{1}-: now also U2.15 (D_{2}-); no longer U2.11 (D_{1}-)
- net D_{2}+: now also U2.12 (D_{1}+); no longer U2.16 (D_{2}+)
- net D_{2}-: now also U2.11 (D_{1}-); no longer U2.15 (D_{2}-)
- net GND: now also U2.27 (TSTPLL/48MCLK), U2.28 (GND), U2.31 (TSTMODE), U2.7 (GND), C4.2, C5.2, C6.2, C8.2, JP1.1 (A), U3.1 (GND), U3.5 (GND)
- net ~OC1: now reaches U2.10 (~OVRCUR1)
- net ~OC1: now also R12.2, U3.16 (~OC1)
- net at U2.13 (~PWRON2): now also U3.4 (~EN2)
- net ~OC2: now reaches U2.14 (~OVRCUR2)
- net ~OC2: now also R13.2, U3.13 (~OC2)
- net at U2.17 (~PWRON3): now also U3.7 (~EN3)
- net ~OC3: now reaches U2.18 (~OVRCUR3)
- net ~OC3: now also R14.2, U3.12 (~OC3)
- net at U2.21 (~PWRON4): now also U3.8 (~EN4)
- net ~OC4: now reaches U2.22 (~OVRCUR4)
- net ~OC4: now also R17.2, U3.9 (~OC4)
- net XTAL2: now reaches U2.29 (XTAL2)
- net XTAL2: now also C5.1, TP7.1, Y1.1
- net XTAL1: now reaches U2.30 (XTAL1)
- net XTAL1: now also C6.1, TP6.1, Y1.2
- net SUSPND: now reaches U2.32 (SUSPND)
- net SUSPND: now also TP5.1
- net ~Reset: now reaches U2.4 (~RESET)
- net ~Reset: now also C4.1, R11.2
- net at U2.6 (EE_{DATA}): now also JP1.2 (C)
- net at U2.9 (~PWRON1): now also U3.3 (~EN1)
- net USB_{D+} renamed USB_D+
- net USB_{D-} renamed USB_D-
- new net PWR_{1}: U3.15 (OUT1)
- new net PWR_{2}: U3.14 (OUT2)
- new net PWR_{3}: U3.10 (OUT4)
- new net PWR_{4}: U3.11 (OUT3)
Other:
- note added: "Ganged vs Individual Overcurrent Protection see datasheet (pg. 4) Should default to low"
- note added: "Pull Up Resistors and Test Points for Overcurrent Signals"
- note removed: "TODO: figure out these signals"
- moved on the sheet: C7, J14, Module1B, U2
