File: usb_mux.kicad_sch (KiCad schematic)
At the start: 17 parts, among them U6 TUSB2046IBVF, U9 TPS2044BD, Y2 HC49USM-FF3F18-6.000MHZ

Commit message: migrated computers
Connections:
- net ~OC1 renamed ~{OC1}
- net ~OC2 renamed ~{OC2}
- net ~OC3 renamed ~{OC3}
- net ~OC4 renamed ~{OC4}
- net ~Reset renamed ~{Reset}
