File: BikeMan.kicad_pcb (KiCad board)
At the start: 2 copper layers, 152.4 x 127 mm, 78 parts, among them J1 Barrel_Jack, J11 PushConnector_8pos, J14 PushConnector_8pos, J8 Conn_01x06_Female, Q1 AUIRF7316QTR, Q2 AUIRF7316QTR, Q3 AUIRF7316QTR, Q4 AUIRF7316QTR, Q5 DMN62D0U-7, Q6 DMN62D0U-7, U1 AP64501, U10 PCF8574DWR, U2 MCP2551, U4 TCN75, U5 MCP2515, U7 PCF85063A, U8 NPIC6C596ADJ, Y1 ABLS7M-16.000MHZ-B-2-T, Y3 Crystal-CM7V-T1A-32.768kHz

Commit message: layout sketching
Parts:
- removed J8: Conn_01x06_Female, Connector_PinSocket_2.54mm:PinSocket_2x03_P2.54mm_Vertical
- added C10: C, Capacitor_SMD:C_0805_2012Metric, F.Cu at (192.5, 96.9)
- added C11: C, Capacitor_SMD:C_0805_2012Metric, F.Cu at (197.0, 96.9)
- added C5: C, Capacitor_SMD:C_0805_2012Metric, F.Cu at (207.3, 167.8)
- added C6: C, Capacitor_SMD:C_0805_2012Metric, F.Cu at (211.3, 164.3)
- added C8: C, Capacitor_SMD:C_0805_2012Metric, F.Cu at (200.2, 171.0)
- added C9: C, Capacitor_SMD:C_0805_2012Metric, F.Cu at (192.5, 99.9)
- added D10: LED_Green, LED_SMD:LED_0805_2012Metric_Pad1.15x1.40mm_HandSolder, F.Cu at (211.5, 161.3)
- added D11: LED_Green, LED_SMD:LED_0805_2012Metric_Pad1.15x1.40mm_HandSolder, F.Cu at (253.3, 72.2)
- added D4: LED_Green, LED_SMD:LED_0805_2012Metric_Pad1.15x1.40mm_HandSolder, F.Cu at (202.7, 167.8)
- added J2: Conn_01x06_Male, Connector_PinHeader_2.54mm:PinHeader_2x03_P2.54mm_Vertical, F.Cu at (164.4, 133.7)
- added J3: Conn_01x06_Male, Connector_PinHeader_2.54mm:PinHeader_2x03_P2.54mm_Vertical, F.Cu at (85.8, 83.1)
- added J4: MicroUSB, ecafe-racer:USB_Micro-B_Amphenol_10104110_Horizontal, F.Cu at (87.6, 123.2)
- added JP10: SolderJumper_2_Open, Jumper:SolderJumper-2_P1.3mm_Open_RoundedPad1.0x1.5mm, F.Cu at (216.1, 164.5)
- added JP7: SolderJumper_3_Open, Jumper:SolderJumper-3_P1.3mm_Open_RoundedPad1.0x1.5mm_NumberLabels, F.Cu at (226.1, 165.1)
- added JP8: SolderJumper_3_Open, Jumper:SolderJumper-3_P1.3mm_Open_RoundedPad1.0x1.5mm_NumberLabels, F.Cu at (226.1, 161.6)
- added JP9: SolderJumper_2_Open, Jumper:SolderJumper-2_P1.3mm_Open_RoundedPad1.0x1.5mm, F.Cu at (209.0, 171.1)
- added Q7: DMN62D0U-7, Package_TO_SOT_SMD:SOT-23, F.Cu at (195.5, 171.7)
- added R11: R, Resistor_SMD:R_0805_2012Metric, F.Cu at (247.7, 72.0)
- added R12: R, Resistor_SMD:R_0805_2012Metric, F.Cu at (247.7, 69.0)
- added R14: R, Resistor_SMD:R_0805_2012Metric, F.Cu at (256.5, 69.0)
- added R16: R, Resistor_SMD:R_0805_2012Metric, F.Cu at (252.1, 74.9)
- added R6: R, Resistor_SMD:R_0805_2012Metric, F.Cu at (216.0, 161.2)
- added R7: R, Resistor_SMD:R_0805_2012Metric, F.Cu at (204.6, 170.8)
- added R8: R, Resistor_SMD:R_0805_2012Metric, F.Cu at (211.7, 167.3)
- added R9: R, Resistor_SMD:R_0805_2012Metric, F.Cu at (247.7, 74.9)
- added U3: MCP2221A, Package_SO:TSSOP-14_4.4x5mm_P0.65mm, F.Cu at (96.5, 123.2)
- added U6: ESP32, ecafe-racer:MODULE_ESP32-WROOM-32, F.Cu at (149.9, 132.1)
- added U9: TPS79933, Package_TO_SOT_SMD:SOT-23-5, F.Cu at (106.7, 121.9)
- Q5, Q6, R21, R22, R23, R24, R25, R26, U10: moved to F.Cu
- R13, R15: value CTS-766161102GP -> R; footprint Package_SO:SOIC-16_3.9x9.9mm_P1.27mm -> Resistor_SMD:R_0805_2012Metric
- moved C15 212.2 mm to (298.3, 10.0)
- moved C16 212.2 mm to (304.8, 5.54)
- moved C17 212.2 mm to (304.8, -0.46)
- moved C18 212.2 mm to (298.9, 3.37)
- moved R10 212.2 mm to (298.3, 10.0)
- moved Y1 212.2 mm to (304.8, 2.54)
- moved TP1 205.2 mm to (280.7, 50.8)
- moved TP2 205.2 mm to (284.2, 50.8)
- moved H3 193.6 mm to (36.8, 53.3)
- moved H4 181.9 mm to (21.6, 48.3)
- moved TP7 176.4 mm to (273.3, 49.5)
- moved TP8 176.4 mm to (273.3, 45.5)
- moved TP3 173.4 mm to (270.8, 53.3)
- moved TP4 173.4 mm to (274.3, 53.3)
- moved TP5 172.2 mm to (277.2, 58.5)
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Connections:
- D5 pad 1: /GPIO/Input_{5} -> /BUS.PWR_{OUT}
- D5 pad 2: /GPIO/I_{5} -> +12V
- D6 pad 1: /GPIO/Input_{8} -> /Input_{3}
- D6 pad 2: /GPIO/I_{8} -> /GPIO/In_{4}
- D7 pad 1: /GPIO/Input_{6} -> +12V
- D7 pad 2: /GPIO/I_{6} -> /BUS.PWR_{IN}
- D8 pad 1: /GPIO/Input_{7} -> /Input_{4}
- D8 pad 2: /GPIO/I_{7} -> /GPIO/In_{3}
- J11 pad 1: /GPIO/Input_{1} -> /BUS.PWR_{IN}
- J11 pad 2: /GPIO/Input_{2} -> /Input_{1}
- J11 pad 3: /GPIO/Input_{3} -> /Input_{2}
- J11 pad 4: /GPIO/Input_{4} -> /Input_{3}
- J11 pad 5: /GPIO/Input_{5} -> /Input_{4}
- J11 pad 6: /GPIO/Input_{6} -> GND
- J11 pad 7: /GPIO/Input_{7} -> /CAN_{L}
- J11 pad 8: /GPIO/Input_{8} -> /CAN_{H}
- J14 pad 1: /GPIO/OUT_{1} -> /BUS.PWR_{OUT}
- J14 pad 2: /GPIO/OUT_{2} -> /GPIO/OUT_{1}
- J14 pad 3: /GPIO/OUT_{3} -> /GPIO/OUT_{2}
- J14 pad 4: /GPIO/OUT_{4} -> /GPIO/OUT_{3}
- J14 pad 5: /GPIO/OUT_{5} -> /GPIO/OUT_{4}
- J14 pad 6: /GPIO/OUT_{6} -> /GPIO/OUT_{5}
- J14 pad 7: /GPIO/OUT_{7} -> /GPIO/OUT_{6}
- J14 pad 8: /GPIO/OUT_{8} -> /GPIO/OUT_{7}
- R13 pad 1: +5V -> /GPIO/In_{2}
- R13 pad 2: +5V -> GND
- R15 pad 1: /GPIO/Input_{1} -> +5V
- R15 pad 2: /GPIO/Input_{2} -> /GPIO/In_{4}
- U10 pad 10: /GPIO/I_{6} -> unconnected-(U10-Pad10)
- U10 pad 11: /GPIO/I_{7} -> unconnected-(U10-Pad11)
- U10 pad 12: /GPIO/I_{8} -> unconnected-(U10-Pad12)
- U10 pad 9: /GPIO/I_{5} -> unconnected-(U10-Pad9)
- U8 pad 14: /GPIO/OUT_CTL_{8} -> /GPIO/SHIFT_IND
Routing:
- net /CAN_{L}: track 87.7 -> 7.62 mm, vias 4 -> 0
- net +5V: track 79.5 -> 2.05 mm, vias 9 -> 0
- net /SDA_{5V}: track 68.8 -> 0.00 mm, vias 3 -> 0
- net /SCL_{5V}: track 68.1 -> 0.00 mm, vias 3 -> 0
- net /CAN_{H}: track 75.6 -> 7.62 mm, vias 3 -> 0
- net /GPIO/OUT_CTL_{8}: track 59.4 -> 0.00 mm, vias 1 -> 0
- net +3V3: track 55.8 -> 0.00 mm, vias 2 -> 0
- net /GPIO/OUT_CTL_{7}: track 54.1 -> 0.00 mm, vias 1 -> 0
- net /SPI.CLK: track 50.1 -> 0.00 mm
- net /SPI.MOSI: track 48.8 -> 0.00 mm
- net /SPI.MISO: track 47.3 -> 0.00 mm
- net /GPIO/OUT_CTL_{6}: track 47.2 -> 0.00 mm, vias 1 -> 0
- net GND: track 56.0 -> 9.12 mm, vias 20 -> 1
- net /SPI.~{CS_{CAN}}: track 45.8 -> 0.00 mm
- net /GPIO/OUT_CTL_{5}: track 41.8 -> 0.00 mm, vias 1 -> 0
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Other:
- board outline removed

Commit message: components group and placed in roughly the right position
Parts:
- removed JP3: SolderJumper_3_Open, Jumper:SolderJumper-3_P1.3mm_Open_RoundedPad1.0x1.5mm_NumberLabels
- added C13: C, Capacitor_SMD:C_0805_2012Metric, F.Cu at (90.7, 110.5)
- added C14: C, Capacitor_SMD:C_0805_2012Metric, F.Cu at (106.9, 96.8)
- added C25: 100uF, Capacitor_SMD:CP_Elec_6.3x5.9, F.Cu at (134.4, 103.9)
- added D12: LED_Green, LED_SMD:LED_0805_2012Metric_Pad1.15x1.40mm_HandSolder, F.Cu at (130.2, 68.6)
- added D13: LED_Green, LED_SMD:LED_0805_2012Metric_Pad1.15x1.40mm_HandSolder, F.Cu at (127.6, 68.6)
- added D14: LED_Green, LED_SMD:LED_0805_2012Metric_Pad1.15x1.40mm_HandSolder, F.Cu at (125.1, 68.6)
- added D15: LED_Green, LED_SMD:LED_0805_2012Metric_Pad1.15x1.40mm_HandSolder, F.Cu at (132.7, 68.6)
- added D16: Diode, Diode_SMD:D_SOD-123F, F.Cu at (160.0, 125.5)
- added R17: R, Resistor_SMD:R_0805_2012Metric, B.Cu at (130.2, 68.6)
- added R18: R, Resistor_SMD:R_0805_2012Metric, B.Cu at (127.6, 68.6)
- added R20: R, Resistor_SMD:R_0805_2012Metric, B.Cu at (125.1, 68.6)
- added R27: R, Resistor_SMD:R_0805_2012Metric, B.Cu at (132.7, 68.6)
- C12, C16, C17, C18, C7: moved to F.Cu
- C5, C8, R11, R13, R14, R15, R7, R8: moved to B.Cu
- moved C16 234.3 mm to (85.1, 86.9)
- moved C17 233.1 mm to (88.7, 86.9), turned to 0 degrees
- moved Y1 232.2 mm to (86.9, 83.0), turned to 90 degrees
- moved C18 223.3 mm to (97.3, 99.4)
- moved C15 222.0 mm to (96.5, 102.6)
- moved R10 222.0 mm to (96.5, 102.6)
- moved Y3 162.3 mm to (84.8, 113.2), turned to 180 degrees
- moved BT1 160.4 mm to (91.1, 128.8), turned to 0 degrees
- moved U7 156.7 mm to (90.9, 114.5), turned to 0 degrees
- moved R14 145.7 mm to (111.0, 60.8), turned to -90 degrees
- moved JP7 145.3 mm to (107.3, 81.3)
- moved D9 144.7 mm to (98.0, 112.5), turned to 180 degrees
- moved JP8 142.3 mm to (106.0, 85.1)
- moved R15 138.8 mm to (113.7, 60.8), turned to -90 degrees
- moved H2 136.5 mm to (165.6, 71.1)
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Connections:
- net /MicroController/CAN_{Rx} renamed /CAN.RX
- net /MicroController/CAN_{Tx} renamed /CAN.TX
- D11 pad 1: GND -> Net-(D11-Pad1)
- D11 pad 2: Net-(D11-Pad2) -> /GPIO/SHIFT_IND
- D6 pad 2: /GPIO/In_{4} -> /GPIO/In_{3}
- D8 pad 2: /GPIO/In_{3} -> /GPIO/In_{4}
- J4 pad 1: unconnected-(J4-Pad1) -> /USB.PWR
- J4 pad 2: unconnected-(J4-Pad2) -> /USB.-
- J4 pad 3: unconnected-(J4-Pad3) -> /USB.+
- J4 pad 5: unconnected-(J4-Pad5) -> GND
- J4 pad 6: unconnected-(J4-Pad6) -> GND
- JP10 pad 2: /MicroController/SCL -> /SCL_{3.3V}
- JP9 pad 2: /MicroController/SDA -> /SDA_{3.3V}
- R14 pad 2: /GPIO/In_{3} -> /GPIO/In_{4}
- R15 pad 2: /GPIO/In_{4} -> /GPIO/In_{3}
- R16 pad 1: /GPIO/SHIFT_IND -> Net-(D11-Pad1)
- R16 pad 2: Net-(D11-Pad2) -> GND
- U10 pad 10: unconnected-(U10-Pad10) -> /GPIO/IND_{3}
- U10 pad 11: unconnected-(U10-Pad11) -> /GPIO/IND_{2}
- U10 pad 12: unconnected-(U10-Pad12) -> /GPIO/IND_{1}
- U10 pad 4: /GPIO/I_{4} -> /GPIO/In_{1}
- U10 pad 5: /GPIO/I_{3} -> /GPIO/In_{2}
- U10 pad 6: /GPIO/I_{2} -> /GPIO/In_{3}
- U10 pad 7: /GPIO/I_{1} -> /GPIO/In_{4}
- U10 pad 9: unconnected-(U10-Pad9) -> /GPIO/IND_{4}
- U3 pad 12: /MicroController/USB_{-} -> /USB.-
- U3 pad 13: /MicroController/USB_{+} -> /USB.+
- U4 pad 5: Net-(JP3-Pad2) -> GND
- U6 pad 10: /MicroController/SPI.CLK -> /SPI.CLK
- U6 pad 11: /MicroController/~{SPI.CS_{CAN}} -> /SPI.~{CS_{CAN}}
- U6 pad 12: /MicroController/~{INT_{CAN}} -> /~{INT_{CAN}}
- U6 pad 26: /MicroController/~{GPIO_{OE}} -> /~{GPIO_{OE}}
- U6 pad 27: /MicroController/~{GPIO_{RS}} -> /~{GPIO_{RS}}
- U6 pad 28: /MicroController/GPIO_{DATA} -> /GPIO_{DATA}
- U6 pad 29: /MicroController/GPIO_{SCLK} -> /GPIO_{sCLK}
- U6 pad 30: /MicroController/GPIO_{RCLK} -> /GPIO_{rCLK}
- U6 pad 36: /MicroController/SCL -> /SCL_{3.3V}
- U6 pad 37: /MicroController/SDA -> /SDA_{3.3V}
- U6 pad 8: /MicroController/SPI.MISO -> /SPI.MISO
- U6 pad 9: /MicroController/SPI.MOSI -> /SPI.MOSI
- U8 pad 11: /GPIO/OUT_CTL_{5} -> /GPIO/OUT_CTL_{7}
- U8 pad 13: /GPIO/OUT_CTL_{7} -> /GPIO/OUT_CTL_{5}
- U8 pad 3: /GPIO/OUT_CTL_{1} -> /GPIO/OUT_CTL_{4}
- U8 pad 4: /GPIO/OUT_CTL_{2} -> /GPIO/OUT_CTL_{3}
- U8 pad 5: /GPIO/OUT_CTL_{3} -> /GPIO/OUT_CTL_{2}
- U8 pad 6: /GPIO/OUT_CTL_{4} -> /GPIO/OUT_CTL_{1}
- U9 pad 3: /Power Supply/enable -> +5V
Routing:
- net GND: track 9.12 -> 56.5 mm, vias 1 -> 14
- net +5V: track 2.05 -> 49.1 mm, vias 0 -> 4
- net /CAN_{L}: track 7.62 -> 41.3 mm, vias 0 -> 3
- net /CAN_{H}: track 7.62 -> 40.1 mm, vias 0 -> 3
- net /GPIO/OUT_CTL_{7}: track 0.00 -> 26.5 mm, vias 0 -> 1
- net /GPIO/OUT_CTL_{1}: track 0.00 -> 23.5 mm, vias 0 -> 1
- net /GPIO/OUT_CTL_{6}: track 0.00 -> 21.6 mm, vias 0 -> 1
- net /GPIO/OUT_CTL_{2}: track 0.00 -> 21.4 mm, vias 0 -> 1
- net /GPIO/OUT_CTL_{5}: track 0.00 -> 20.3 mm, vias 0 -> 1
- net /GPIO/OUT_CTL_{4}: track 0.00 -> 19.9 mm, vias 0 -> 1
- net /GPIO/OUT_CTL_{3}: track 0.00 -> 18.6 mm, vias 0 -> 1
- net +3V3: track 0.00 -> 18.4 mm, vias 0 -> 2
- net Net-(JP8-Pad2): track 0.00 -> 15.5 mm, vias 0 -> 2
- net /CAN Peripherals/CAN_{RxLOW}: track 0.00 -> 13.1 mm
- net /CAN Peripherals/OSC2: track 0.00 -> 8.43 mm
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- removed copper zone on F.Cu, net +3V3
- removed copper zone on B.Cu, net +5V
- removed copper zone on F.Cu, net /Power Supply/PWR_IN
Other:
- board outline added: 89.8 x 100.5 mm

Commit message: WIP
Parts:
- added D17: LED_Green, LED_SMD:LED_0805_2012Metric_Pad1.15x1.40mm_HandSolder, F.Cu at (135.5, 68.5)
- added JP3: Jumper_2_Open, Connector_PinHeader_2.54mm:PinHeader_1x02_P2.54mm_Vertical, F.Cu at (181.8, 118.5)
- added R28: R, Resistor_SMD:R_0805_2012Metric, F.Cu at (186.3, 117.7)
- added R29: R, Resistor_SMD:R_0805_2012Metric, B.Cu at (135.5, 68.5)
- moved J2 46.7 mm to (160.3, 152.3), turned to 180 degrees
- moved D10 29.4 mm to (102.0, 131.6), turned to 90 degrees
- moved R8 29.4 mm to (102.0, 131.6), turned to 90 degrees
- moved Q5 16.5 mm to (112.6, 99.4)
- moved Q6 16.5 mm to (116.3, 99.4)
- moved R21 16.5 mm to (113.3, 102.9)
- moved R22 16.5 mm to (113.3, 95.8)
- moved R23 16.5 mm to (115.5, 102.9)
- moved R24 16.5 mm to (115.5, 95.8)
- moved JP10 12.9 mm to (154.6, 128.0)
- moved C14 11.7 mm to (110.5, 85.7)
- moved JP6 11.7 mm to (115.1, 81.6)
- moved U4 11.7 mm to (114.6, 87.2)
- moved C9 10.7 mm to (138.6, 104.1)
- moved C10 10.7 mm to (142.2, 107.2)
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Connections:
- net /GPIO/OUT_{8} renamed /GPIO/OUT_IND
- D10 pad 1: GND -> Net-(R8-Pad1)
- D10 pad 2: Net-(D10-Pad2) -> /MicroController/mcu_indicator
- D4 pad 1: GND -> Net-(R7-Pad1)
- D4 pad 2: Net-(D4-Pad2) -> /MicroController/usb_indicator
- J14 pad 1: /BUS.PWR_{OUT} -> /GPIO/OUT_{1}
- J14 pad 2: /GPIO/OUT_{1} -> /GPIO/OUT_{2}
- J14 pad 3: /GPIO/OUT_{2} -> /GPIO/OUT_{3}
- J14 pad 4: /GPIO/OUT_{3} -> /GPIO/OUT_{4}
- J14 pad 5: /GPIO/OUT_{4} -> /GPIO/OUT_{5}
- J14 pad 6: /GPIO/OUT_{5} -> /GPIO/OUT_{6}
- J14 pad 7: /GPIO/OUT_{6} -> /GPIO/OUT_{7}
- J14 pad 8: /GPIO/OUT_{7} -> /BUS.PWR_{OUT}
- JP7 pad 3: /CAN Peripherals/CAN_{Rx}DIR -> /CAN.RX
- JP8 pad 3: /CAN Peripherals/CAN_{Tx}DIR -> /CAN.TX
- Q1 pad 2: /GPIO/OUT_CTL_{8} -> /GPIO/OUT_CTL_{7}
- R19 pad 9: /GPIO/OUT_CTL_{8} -> /GPIO/OUT_CTL_{7}
- R7 pad 1: /MicroController/usb_indicator -> Net-(R7-Pad1)
- R7 pad 2: Net-(D4-Pad2) -> GND
- R8 pad 1: /MicroController/mcu_indicator -> Net-(R8-Pad1)
- R8 pad 2: Net-(D10-Pad2) -> GND
- U6 pad 10: /SPI.CLK -> /GPIO_{DATA}
- U6 pad 11: /SPI.~{CS_{CAN}} -> /~{GPIO_{RS}}
- U6 pad 12: /~{INT_{CAN}} -> /~{GPIO_{OE}}
- U6 pad 26: /~{GPIO_{OE}} -> /SPI.~{CS_{CAN}}
- U6 pad 27: /~{GPIO_{RS}} -> /SPI.MISO
- U6 pad 28: /GPIO_{DATA} -> /SPI.MOSI
- U6 pad 29: /GPIO_{sCLK} -> /SPI.CLK
- U6 pad 30: /GPIO_{rCLK} -> /~{INT_{CAN}}
- U6 pad 33: unconnected-(U6-Pad33) -> /MicroController/mcu_indicator
- U6 pad 8: /SPI.MISO -> /GPIO_{rCLK}
- U6 pad 9: /SPI.MOSI -> /GPIO_{sCLK}
Routing:
- net +5V: track 49.1 -> 122.1 mm, vias 4 -> 5
- net /CAN.RX: track 0.00 -> 56.3 mm
- net /CAN.TX: track 0.00 -> 51.4 mm
- net /~{INT_{CAN}}: track 0.00 -> 35.4 mm
- net /SPI.CLK: track 0.00 -> 33.8 mm
- net /SPI.MOSI: track 0.00 -> 32.2 mm
- net /SPI.MISO: track 0.00 -> 30.6 mm
- net Net-(BT1-Pad1): track 0.00 -> 30.3 mm, vias 0 -> 2
- net /SPI.~{CS_{CAN}}: track 0.00 -> 28.9 mm
- net /MicroController/bootmode_select: track 0.00 -> 28.5 mm, vias 0 -> 2
- net GND: track 56.5 -> 84.5 mm, vias 14 -> 23
- net /SDA_{5V}: track 2.02 -> 29.8 mm, vias 0 -> 3
- net /MicroController/esp_rx: track 0.00 -> 27.6 mm
- net /MicroController/esp_tx: track 0.00 -> 27.4 mm
- net /SCL_{5V}: track 2.02 -> 29.0 mm, vias 0 -> 3
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Other:
- board size 89.8 x 100.5 mm -> 90 x 99 mm

Commit message: WIP
Parts:
- added D18: LED_Green, LED_SMD:LED_0805_2012Metric_Pad1.15x1.40mm_HandSolder, F.Cu at (121.1, 60.0)
- added D19: LED_Green, LED_SMD:LED_0805_2012Metric_Pad1.15x1.40mm_HandSolder, F.Cu at (150.2, 96.8)
- added R30: R, Resistor_SMD:R_0805_2012Metric, B.Cu at (121.1, 60.0)
- added R31: R, Resistor_SMD:R_0805_2012Metric, B.Cu at (150.2, 96.8)
- R16, R28: moved to B.Cu
- moved D11 12.9 mm to (148.4, 82.8)
- moved R16 11.9 mm to (148.4, 82.8)
- moved R28 2.80 mm to (185.2, 120.2), turned to 90 degrees
- moved D12 2.05 mm to (129.2, 66.8)
- moved D13 2.05 mm to (126.7, 66.8)
- moved D15 2.05 mm to (131.8, 66.8)
- moved D17 2.05 mm to (134.6, 66.7)
- moved R17 2.05 mm to (129.2, 66.8)
- moved R18 2.05 mm to (126.7, 66.8)
- moved R27 2.05 mm to (131.8, 66.8)
- moved R29 2.05 mm to (134.6, 66.7)
- moved D14 2.05 mm to (124.2, 66.8)
- moved R20 2.05 mm to (124.2, 66.8)
- moved D7 0.62 mm to (124.2, 59.9)
Connections:
- D12 pad 2: /GPIO/IND_{1} -> /GPIO/IND_{2}
- D13 pad 2: /GPIO/IND_{2} -> /GPIO/IND_{3}
- D14 pad 2: /GPIO/IND_{3} -> /GPIO/IND_{4}
- D15 pad 2: /GPIO/IND_{4} -> /GPIO/IND_{1}
- U6 pad 10: /GPIO_{DATA} -> /~{GPIO_{RS}}
- U6 pad 11: /~{GPIO_{RS}} -> /GPIO_{rCLK}
- U6 pad 8: /GPIO_{rCLK} -> /GPIO_{sCLK}
- U6 pad 9: /GPIO_{sCLK} -> /GPIO_{DATA}
Routing:
- net /GPIO_{DATA}: track 1.96 -> 93.5 mm, vias 1 -> 2
- net /~{GPIO_{RS}}: track 1.96 -> 90.4 mm, vias 1 -> 2
- net /~{GPIO_{OE}}: track 1.96 -> 88.5 mm, vias 1 -> 2
- net /GPIO_{sCLK}: track 0.00 -> 83.4 mm
- net /GPIO_{rCLK}: track 0.00 -> 78.4 mm
- net /SCL_{3.3V}: track 24.4 -> 50.4 mm, vias 1 -> 4
- net /SDA_{3.3V}: track 22.5 -> 47.5 mm, vias 0 -> 4
- net /GPIO/IND_{1}: track 0.00 -> 23.0 mm
- net /GPIO/IND_{2}: track 0.00 -> 21.8 mm
- net /GPIO/IND_{3}: track 0.00 -> 20.6 mm
- net /GPIO/IND_{4}: track 0.00 -> 19.3 mm
- net +12V: track 19.0 -> 35.0 mm, vias 8 -> 9
- net /BUS.PWR_{IN}: track 7.62 -> 17.7 mm
- net /BUS.PWR_{OUT}: track 7.62 -> 13.9 mm
- net Net-(D18-Pad1): track 0.00 -> 3.66 mm, vias 0 -> 1
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
Commit message: WIP
Parts:
- added R32: R, Resistor_SMD:R_0805_2012Metric, B.Cu at (151.8, 127.0)
- added R33: R, Resistor_SMD:R_0805_2012Metric, B.Cu at (151.8, 129.0)
- added R34: R, Resistor_SMD:R_0805_2012Metric, B.Cu at (151.8, 131.0)
- J2: value Conn_01x06_Male -> Conn_01x12_Male; footprint Connector_PinHeader_2.54mm:PinHeader_2x03_P2.54mm_Vertical -> Connector_PinHeader_2.54mm:PinHeader_2x06_P2.54mm_Vertical
- moved JP3 46.8 mm to (135.0, 115.5)
- moved R28 46.8 mm to (138.5, 117.2)
- moved J2 31.5 mm to (155.7, 121.2), turned to 0 degrees
- moved C25 27.2 mm to (141.0, 126.0), turned to 90 degrees
- moved C1 26.9 mm to (139.3, 87.9)
- moved C19 26.9 mm to (135.9, 99.4)
- moved C2 26.9 mm to (138.1, 99.5)
- moved C20 26.9 mm to (130.8, 91.6)
- moved C21 26.9 mm to (140.2, 99.4)
- moved C22 26.9 mm to (138.0, 99.4)
- moved C23 26.9 mm to (138.6, 95.4)
- moved C3 26.9 mm to (142.3, 92.9)
- moved C4 26.9 mm to (130.7, 86.1)
- moved JP2 26.9 mm to (130.9, 89.3)
- moved L1 26.9 mm to (129.6, 96.6)
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Connections:
- J2 pad 1: /MicroController/esp_tx -> unconnected-(J2-Pad1)
- J2 pad 2: /MicroController/esp_rx -> +5V
- J2 pad 3: /MicroController/~esp_reset -> /SDA_{3.3V}
- J2 pad 4: /MicroController/bootmode_select -> +5V
- J2 pad 5: /MicroController/~silent_boot -> /SCL_{3.3V}
Routing:
- net /SDA_{3.3V}: track 47.5 -> 116.3 mm
- net /SCL_{3.3V}: track 50.4 -> 115.8 mm
- net /MicroController/esp_tx: track 27.4 -> 68.5 mm
- net /MicroController/esp_rx: track 27.6 -> 66.3 mm
- net +5V: track 122.1 -> 151.3 mm, vias 5 -> 7
- net +3V3: track 20.8 -> 49.3 mm
- net GND: track 84.5 -> 99.7 mm, vias 23 -> 25
- net /GPIO/SHIFT_IND: track 0.00 -> 12.7 mm, vias 0 -> 2
- net /USB.-: track 0.00 -> 7.31 mm
- net /USB.+: track 0.00 -> 7.21 mm
- net +12V: track 35.0 -> 40.5 mm, vias 9 -> 15
- net Net-(JP9-Pad1): track 8.28 -> 4.95 mm
- net /MicroController/usb_indicator: track 0.00 -> 2.92 mm
- net Net-(R7-Pad1): track 0.00 -> 2.71 mm, vias 0 -> 1
- net Net-(JP10-Pad1): track 7.29 -> 6.21 mm
- added copper zone on F.Cu, net /Power Supply/PWR_IN
Other:
- board text added: "Dennis v0.2"
- board text removed: "Dennis v0.1.3"
