File: BikeMan.kicad_sch (KiCad schematic)
At the start: 17 parts, among them J11 PushConnector_8pos, J14 PushConnector_8pos, J3 Conn_01x06_Male, J4 MicroUSB, Q5 DMN62D0U-7, Q6 DMN62D0U-7

Commit message: WIP
Parts:
- added D?: LED_Green, LED_SMD:LED_0805_2012Metric_Pad1.15x1.40mm_HandSolder, symbol ecafe-racer:LED_Green
- added R?: R, Resistor_SMD:R_0805_2012Metric, symbol Device:R
Connections:
- net BUS.PWR_{IN}: now also D?.2
- net BUS.PWR_{OUT}: now also J14.8 (Pin_8); no longer J14.1 (Pin_1)
- net GND: now also R?.2
- net GPIO/OUT_{1}: now also J14.1 (Pin_1); no longer J14.2 (Pin_2)
- net GPIO/OUT_{2}: now also J14.2 (Pin_2); no longer J14.3 (Pin_3)
- net GPIO/OUT_{3}: now also J14.3 (Pin_3); no longer J14.4 (Pin_4)
- net GPIO/OUT_{4}: now also J14.4 (Pin_4); no longer J14.5 (Pin_5)
- net GPIO/OUT_{5}: now also J14.5 (Pin_5); no longer J14.6 (Pin_6)
- net GPIO/OUT_{6}: now also J14.6 (Pin_6); no longer J14.7 (Pin_7)
- net GPIO/OUT_{7}: now also J14.7 (Pin_7); no longer J14.8 (Pin_8)
- new net: D?.1, R?.1
Other:
- sheet CAN Peripherals ports: added CAN_{Rx}DIR, CAN_{Tx}DIR; removed none
- note added: "Bus Power Indicator"
- moved on the sheet: J14

Commit message: WIP
Parts:
- gave numbers to parts that had none: 2
Changed lines of the file:
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@@
     (stroke (width 0) (type solid) (color 0 0 0 0))
   )
-  (bus (pts (xy 165.1 87.63) (xy 165.1 118.11))
+  (bus (pts (xy 165.1 85.09) (xy 165.1 118.11))
     (stroke (width 0) (type solid) (color 0 0 0 0))
   )
-  (bus (pts (xy 168.91 72.39) (xy 168.91 121.92))
+  (bus (pts (xy 168.91 69.85) (xy 168.91 121.92))
     (stroke (width 0) (type solid) (color 0 0 0 0))
   )
@@
   (symbol (lib_id "power:GND") (at 133.35 193.04 0) (unit 1)
     (in_bom yes) (on_board yes) (fields_autoplaced)
-    (property "Reference" "#PWR?" (id 0) (at 133.35 199.39 0)
+    (property "Reference" "#PWR0146" (id 0) (at 133.35 199.39 0)
       (effects (font (size 1.27 1.27)) hide)
     )
@@
   (symbol (lib_id "Device:R") (at 133.35 189.23 0) (unit 1)
     (in_bom yes) (on_board yes) (fields_autoplaced)
-    (property "Reference" "R?" (id 0) (at 135.89 187.9599 0)
+    (property "Reference" "R30" (id 0) (at 135.89 187.9599 0)
       (effects (font (size 1.27 1.27)) (justify left))
     )
@@
   (symbol (lib_id "ecafe-racer:LED_Green") (at 133.35 181.61 90) (unit 1)
     (in_bom yes) (on_board yes) (fields_autoplaced)
-    (property "Reference" "D?" (id 0) (at 137.16 180.5304 90)
+    (property "Reference" "D18" (id 0) (at 137.16 180.5304 90)
       (effects (font (size 1.27 1.27)) (justify right))
     )
@@
       (reference "#PWR0145") (unit 1) (value "GND") (footprint "")
     )
+    (path "/aff81f6a-eb88-48b1-a6a4-5002453e6727"
+      (reference "#PWR0146") (unit 1) (value "GND") (footprint "")
+    )
+    (path "/97a6e0d0-e45e-4fe9-a578-968187c50165/60f00d35-d21b-4e1d-a8f4-81206ed7e8f6"
+      (reference "#PWR0147") (unit 1) (value "GND") (footprint "")
+    )
     (path "/97a6e0d0-e45e-4fe9-a578-968187c50165/fcb0cd51-9f00-497e-9bbc-b2dbab7db47b"
       (reference "#PWR0155") (unit 1) (value "GND") (footprint "")
@@
       (reference "#PWR0199") (unit 1) (value "+5V") (footprint "")
     )
-    (path "/97a6e0d0-e45e-4fe9-a578-968187c50165/60f00d35-d21b-4e1d-a8f4-81206ed7e8f6"
-      (reference "#PWR?") (unit 1) (value "GND") (footprint "")
-    )
-    (path "/aff81f6a-eb88-48b1-a6a4-5002453e6727"
-      (reference "#PWR?") (unit 1) (value "GND") (footprint "")
-    )
     (path "/19c8499b-69ca-41a4-81d4-1e5248b15d37/eeb646f8-ecd2-4f7a-a6bd-d4a25607ff16"
       (reference "BT1") (unit 1) (value "Battery_Cell") (footprint "Battery:BatteryHolder_Keystone_3001_1x12mm")
@@
     )
     (path "/1f0d7149-a7e7-4060-99b7-78d2f8bf29d7"
-      (reference "D?") (unit 1) (value "LED_Green") (footprint "LED_SMD:LED_0805_2012Metric_Pad1.15x1.40mm_HandSolder")
+      (reference "D18") (unit 1) (value "LED_Green") (footprint "LED_SMD:LED_0805_2012Metric_Pad1.15x1.40mm_HandSolder")
     )
     (path "/97a6e0d0-e45e-4fe9-a578-968187c50165/8799ebb8-87c3-448e-921a-a09aa715c0e2"
-      (reference "D?") (unit 1) (value "LED_Green") (footprint "LED_SMD:LED_0805_2012Metric_Pad1.15x1.40mm_HandSolder")
+      (reference "D19") (unit 1) (value "LED_Green") (footprint "LED_SMD:LED_0805_2012Metric_Pad1.15x1.40mm_HandSolder")
     )
     (path "/56031da0-b30d-40e7-9bf7-184fa400b03d"
@@
     )
     (path "/c027a0c7-289c-4bc3-82dc-144d4938cbe1"
-      (reference "R?") (unit 1) (value "R") (footprint "Resistor_SMD:R_0805_2012Metric")
+      (reference "R30") (unit 1) (value "R") (footprint "Resistor_SMD:R_0805_2012Metric")
     )
     (path "/97a6e0d0-e45e-4fe9-a578-968187c50165/c69c0079-f61b-44b3-b944-31f1b9deadad"
-      (reference "R?") (unit 1) (value "R") (footprint "Resistor_SMD:R_0805_2012Metric")
+      (reference "R31") (unit 1) (value "R") (footprint "Resistor_SMD:R_0805_2012Metric")
     )
     (path "/a37aae83-17bc-4ab3-8207-20408c46a8d9/ce1e3873-ad4a-46e4-bc8e-1516017c2b73"

Commit message: WIP
Parts:
- added D?: LED_Green, LED_SMD:LED_0805_2012Metric_Pad1.15x1.40mm_HandSolder, symbol ecafe-racer:LED_Green
- added R?: R, Resistor_SMD:R_0805_2012Metric, symbol Device:R
Connections:
- net GND: now also R?.2
- net USB.PWR: now also D?.2
- new net: D?.1, R?.1
Other:
- note added: "Power Indicators"
- note removed: "Bus Power Indicator"
- moved on the sheet: D18, R30
Changed lines of the file:
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@@
     (stroke (width 0) (type solid) (color 0 0 0 0))
   )
-  (wire (pts (xy 133.35 166.37) (xy 133.35 177.8))
+  (wire (pts (xy 127 166.37) (xy 127 177.8))
+    (stroke (width 0) (type solid) (color 0 0 0 0))
+  )
+  (wire (pts (xy 140.97 166.37) (xy 140.97 177.8))
     (stroke (width 0) (type solid) (color 0 0 0 0))
   )
@@
     (effects (font (size 1.27 1.27)) (justify left bottom))
   )
-  (text "Bus Power Indicator" (at 143.51 191.77 90)
+  (text "Power Indicators" (at 153.67 193.04 90)
     (effects (font (size 1.27 1.27)) (justify left bottom))
   )
@@
     (effects (font (size 1.27 1.27)) (justify right bottom))
   )
-  (label "BUS.PWR_{IN}" (at 133.35 166.37 270)
+  (label "BUS.PWR_{IN}" (at 127 166.37 270)
+    (effects (font (size 1.27 1.27)) (justify right bottom))
+  )
+  (label "USB.PWR" (at 140.97 166.37 270)
     (effects (font (size 1.27 1.27)) (justify right bottom))
   )
@@
     (pin "1")
   )
-  (symbol (lib_id "power:GND") (at 133.35 193.04 0) (unit 1)
+  (symbol (lib_id "power:GND") (at 127 193.04 0) (unit 1)
     (in_bom yes) (on_board yes) (fields_autoplaced)
-    (property "Reference" "#PWR0146" (id 0) (at 133.35 199.39 0)
-      (effects (font (size 1.27 1.27)) hide)
-    )
-    (property "Value" "GND" (id 1) (at 133.35 198.12 0))
-    (property "Footprint" "" (id 2) (at 133.35 193.04 0)
-      (effects (font (size 1.27 1.27)) hide)
-    )
-    (property "Datasheet" "" (id 3) (at 133.35 193.04 0)
+    (property "Reference" "#PWR0146" (id 0) (at 127 199.39 0)
+      (effects (font (size 1.27 1.27)) hide)
+    )
+    (property "Value" "GND" (id 1) (at 127 198.12 0))
+    (property "Footprint" "" (id 2) (at 127 193.04 0)
+      (effects (font (size 1.27 1.27)) hide)
+    )
+    (property "Datasheet" "" (id 3) (at 127 193.04 0)
+      (effects (font (size 1.27 1.27)) hide)
+    )
+    (pin "1")
+  )
+  (symbol (lib_id "power:GND") (at 140.97 193.04 0) (unit 1)
+    (in_bom yes) (on_board yes) (fields_autoplaced)
+    (property "Reference" "#PWR?" (id 0) (at 140.97 199.39 0)
+      (effects (font (size 1.27 1.27)) hide)
+    )
+    (property "Value" "GND" (id 1) (at 140.97 198.12 0))
+    (property "Footprint" "" (id 2) (at 140.97 193.04 0)
+      (effects (font (size 1.27 1.27)) hide)
+    )
+    (property "Datasheet" "" (id 3) (at 140.97 193.04 0)
       (effects (font (size 1.27 1.27)) hide)
     )
@@
     (pin "2")
   )
-  (symbol (lib_id "Device:R") (at 133.35 189.23 0) (unit 1)
+  (symbol (lib_id "Device:R") (at 127 189.23 0) (unit 1)
     (in_bom yes) (on_board yes) (fields_autoplaced)
-    (property "Reference" "R30" (id 0) (at 135.89 187.9599 0)
-      (effects (font (size 1.27 1.27)) (justify left))
-    )
-    (property "Value" "R" (id 1) (at 135.89 190.4999 0)
-      (effects (font (size 1.27 1.27)) (justify left))
-    )
-    (property "Footprint" "Resistor_SMD:R_0805_2012Metric" (id 2) (at 131.572 189.23 90)
-      (effects (font (size 1.27 1.27)) hide)
-    )
-    (property "Datasheet" "~" (id 3) (at 133.35 189.23 0)
+    (property "Reference" "R30" (id 0) (at 129.54 187.9599 0)
+      (effects (font (size 1.27 1.27)) (justify left))
+    )
+    (property "Value" "R" (id 1) (at 129.54 190.4999 0)
+      (effects (font (size 1.27 1.27)) (justify left))
+    )
+    (property "Footprint" "Resistor_SMD:R_0805_2012Metric" (id 2) (at 125.222 189.23 90)
+      (effects (font (size 1.27 1.27)) hide)
+    )
+    (property "Datasheet" "~" (id 3) (at 127 189.23 0)
+      (effects (font (size 1.27 1.27)) hide)
+    )
+    (pin "1")
+    (pin "2")
+  )
+  (symbol (lib_id "Device:R") (at 140.97 189.23 0) (unit 1)
+    (in_bom yes) (on_board yes) (fields_autoplaced)
+    (property "Reference" "R?" (id 0) (at 143.51 187.9599 0)
+      (effects (font (size 1.27 1.27)) (justify left))
+    )
+    (property "Value" "R" (id 1) (at 143.51 190.4999 0)
+      (effects (font (size 1.27 1.27)) (justify left))
+    )
+    (property "Footprint" "Resistor_SMD:R_0805_2012Metric" (id 2) (at 139.192 189.23 90)
+      (effects (font (size 1.27 1.27)) hide)
+    )
+    (property "Datasheet" "~" (id 3) (at 140.97 189.23 0)
       (effects (font (size 1.27 1.27)) hide)
     )
@@
     (pin "1")
   )
-  (symbol (lib_id "ecafe-racer:LED_Green") (at 133.35 181.61 90) (unit 1)
+  (symbol (lib_id "ecafe-racer:LED_Green") (at 127 181.61 90) (unit 1)
     (in_bom yes) (on_board yes) (fields_autoplaced)
-    (property "Reference" "D18" (id 0) (at 137.16 180.5304 90)
-      (effects (font (size 1.27 1.27)) (justify right))
-    )
-    (property "Value" "LED_Green" (id 1) (at 137.16 183.0704 90)
+    (property "Reference" "D18" (id 0) (at 130.81 180.5304 90)
+      (effects (font (size 1.27 1.27)) (justify right))
+    )
+    (property "Value" "LED_Green" (id 1) (at 130.81 183.0704 90)
       (effects (font (size 1.27 1.27)) (justify right) hide)
     )
-    (property "Footprint" "LED_SMD:LED_0805_2012Metric_Pad1.15x1.40mm_HandSolder" (id 2) (at 121.92 172.72 0)
-      (effects (font (size 1.27 1.27)) hide)
-    )
-    (property "Datasheet" "https://vcclite.com/wp-content/uploads/wpallimport/files/files/CMD1721Seriesver3.pdf" (id 3) (at 129.54 177.8 0)
-      (effects (font (size 1.27 1.27)) hide)
-    )
-    (property "Vendor" "Digikey" (id 4) (at 114.3 199.39 0)
-      (effects (font (size 1.27 1.27)) hide)
-    )
-    (property "Vendor Part" "L62405CT-ND" (id 5) (at 116.84 195.58 0)
-      (effects (font (size 1.27 1.27)) hide)
-    )
-    (property "Manufacturer" "Visual Communications Company - VCC" (id 6) (at 124.46 182.88 0)
-      (effects (font (size 1.27 1.27)) hide)
-    )
-    (property "Manufacturer Part" "CMD17-21VGC/TR8" (id 7) (at 119.38 193.04 0)
+    (property "Footprint" "LED_SMD:LED_0805_2012Metric_Pad1.15x1.40mm_HandSolder" (id 2) (at 115.57 172.72 0)
+      (effects (font (size 1.27 1.27)) hide)
+    )
+    (property "Datasheet" "https://vcclite.com/wp-content/uploads/wpallimport/files/files/CMD1721Seriesver3.pdf" (id 3) (at 123.19 177.8 0)
+      (effects (font (size 1.27 1.27)) hide)
+    )
+    (property "Vendor" "Digikey" (id 4) (at 107.95 199.39 0)
+      (effects (font (size 1.27 1.27)) hide)
+    )
+    (property "Vendor Part" "L62405CT-ND" (id 5) (at 110.49 195.58 0)
+      (effects (font (size 1.27 1.27)) hide)
+    )
+    (property "Manufacturer" "Visual Communications Company - VCC" (id 6) (at 118.11 182.88 0)
+      (effects (font (size 1.27 1.27)) hide)
+    )
+    (property "Manufacturer Part" "CMD17-21VGC/TR8" (id 7) (at 113.03 193.04 0)
+      (effects (font (size 1.27 1.27)) hide)
+    )
+    (pin "1")
+    (pin "2")
+  )
+  (symbol (lib_id "ecafe-racer:LED_Green") (at 140.97 181.61 90) (unit 1)
+    (in_bom yes) (on_board yes) (fields_autoplaced)
+    (property "Reference" "D?" (id 0) (at 144.78 180.5304 90)
+      (effects (font (size 1.27 1.27)) (justify right))
+    )
+    (property "Value" "LED_Green" (id 1) (at 144.78 183.0704 90)
+      (effects (font (size 1.27 1.27)) (justify right) hide)
+    )
+    (property "Footprint" "LED_SMD:LED_0805_2012Metric_Pad1.15x1.40mm_HandSolder" (id 2) (at 129.54 172.72 0)
+      (effects (font (size 1.27 1.27)) hide)
+    )
+    (property "Datasheet" "https://vcclite.com/wp-content/uploads/wpallimport/files/files/CMD1721Seriesver3.pdf" (id 3) (at 137.16 177.8 0)
+      (effects (font (size 1.27 1.27)) hide)
+    )
+    (property "Vendor" "Digikey" (id 4) (at 121.92 199.39 0)
+      (effects (font (size 1.27 1.27)) hide)
+    )
+    (property "Vendor Part" "L62405CT-ND" (id 5) (at 124.46 195.58 0)
+      (effects (font (size 1.27 1.27)) hide)
+    )
+    (property "Manufacturer" "Visual Communications Company - VCC" (id 6) (at 132.08 182.88 0)
+      (effects (font (size 1.27 1.27)) hide)
+    )
+    (property "Manufacturer Part" "CMD17-21VGC/TR8" (id 7) (at 127 193.04 0)
       (effects (font (size 1.27 1.27)) hide)
     )
@@
       (reference "#PWR0199") (unit 1) (value "+5V") (footprint "")
     )
+    (path "/57522df6-13d5-49b6-b736-3650cb049fbf"
+      (reference "#PWR?") (unit 1) (value "GND") (footprint "")
+    )
     (path "/19c8499b-69ca-41a4-81d4-1e5248b15d37/eeb646f8-ecd2-4f7a-a6bd-d4a25607ff16"
       (reference "BT1") (unit 1) (value "Battery_Cell") (footprint "Battery:BatteryHolder_Keystone_3001_1x12mm")
@@
       (reference "D19") (unit 1) (value "LED_Green") (footprint "LED_SMD:LED_0805_2012Metric_Pad1.15x1.40mm_HandSolder")
     )
+    (path "/c9ff74f8-0bc9-4f11-a548-132fe582a2f8"
+      (reference "D?") (unit 1) (value "LED_Green") (footprint "LED_SMD:LED_0805_2012Metric_Pad1.15x1.40mm_HandSolder")
+    )
     (path "/56031da0-b30d-40e7-9bf7-184fa400b03d"
       (reference "H1") (unit 1) (value "MountingHole_Pad") (footprint "MountingHole:MountingHole_3.2mm_M3")
@@
       (reference "R34") (unit 1) (value "R") (footprint "Resistor_SMD:R_0805_2012Metric")
     )
+    (path "/802cfdee-6aab-4737-871d-9f7e3f99c57a"
+      (reference "R?") (unit 1) (value "R") (footprint "Resistor_SMD:R_0805_2012Metric")
+    )
     (path "/a37aae83-17bc-4ab3-8207-20408c46a8d9/ce1e3873-ad4a-46e4-bc8e-1516017c2b73"

Commit message: finished routing
Parts:
- gave numbers to parts that had none: 2
Connections:
- net +5V: now also J3.6 (Pin_6); no longer J3.1 (Pin_1)
- net CAN_{L}: now also J3.4 (Pin_4); no longer J3.3 (Pin_3)
- net GND: now also J3.5 (Pin_5); no longer J3.6 (Pin_6)
Other:
- note removed: "I2C Bus?"
Changed lines of the file:
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@@
     (stroke (width 0) (type solid) (color 0 0 0 0))
   )
-  (wire (pts (xy 104.14 181.61) (xy 114.3 181.61))
-    (stroke (width 0) (type solid) (color 0 0 0 0))
-  )
-  (wire (pts (xy 104.14 189.23) (xy 106.68 189.23))
-    (stroke (width 0) (type solid) (color 0 0 0 0))
-  )
-  (wire (pts (xy 106.68 173.99) (xy 106.68 176.53))
-    (stroke (width 0) (type solid) (color 0 0 0 0))
-  )
-  (wire (pts (xy 106.68 176.53) (xy 104.14 176.53))
-    (stroke (width 0) (type solid) (color 0 0 0 0))
-  )
-  (wire (pts (xy 106.68 189.23) (xy 106.68 191.77))
+  (wire (pts (xy 104.14 184.15) (xy 114.3 184.15))
+    (stroke (width 0) (type solid) (color 0 0 0 0))
+  )
+  (wire (pts (xy 104.14 186.69) (xy 106.68 186.69))
+    (stroke (width 0) (type solid) (color 0 0 0 0))
+  )
+  (wire (pts (xy 106.68 186.69) (xy 106.68 194.31))
+    (stroke (width 0) (type solid) (color 0 0 0 0))
+  )
+  (wire (pts (xy 107.95 171.45) (xy 107.95 189.23))
+    (stroke (width 0) (type solid) (color 0 0 0 0))
+  )
+  (wire (pts (xy 107.95 189.23) (xy 104.14 189.23))
     (stroke (width 0) (type solid) (color 0 0 0 0))
   )
@@
     (effects (font (size 1.27 1.27)) (justify left bottom))
   )
-  (text "I2C Bus?" (at 109.855 187.325 0)
-    (effects (font (size 1.27 1.27)) (justify left bottom))
-  )
   (text "Power Indicators" (at 153.67 193.04 90)
     (effects (font (size 1.27 1.27)) (justify left bottom))
@@
     (effects (font (size 1.27 1.27)) (justify right bottom))
   )
-  (label "CAN_{L}" (at 114.3 181.61 180)
+  (label "CAN_{L}" (at 114.3 184.15 180)
     (effects (font (size 1.27 1.27)) (justify right bottom))
   )
@@
     (pin "1")
   )
-  (symbol (lib_id "power:+5V") (at 106.68 173.99 0) (unit 1)
+  (symbol (lib_id "power:+5V") (at 107.95 171.45 0) (unit 1)
     (in_bom yes) (on_board yes) (fields_autoplaced)
-    (property "Reference" "#PWR0124" (id 0) (at 106.68 177.8 0)
-      (effects (font (size 1.27 1.27)) hide)
-    )
-    (property "Value" "+5V" (id 1) (at 106.68 168.91 0))
-    (property "Footprint" "" (id 2) (at 106.68 173.99 0)
-      (effects (font (size 1.27 1.27)) hide)
-    )
-    (property "Datasheet" "" (id 3) (at 106.68 173.99 0)
+    (property "Reference" "#PWR0124" (id 0) (at 107.95 175.26 0)
+      (effects (font (size 1.27 1.27)) hide)
+    )
+    (property "Value" "+5V" (id 1) (at 107.95 166.37 0))
+    (property "Footprint" "" (id 2) (at 107.95 171.45 0)
+      (effects (font (size 1.27 1.27)) hide)
+    )
+    (property "Datasheet" "" (id 3) (at 107.95 171.45 0)
       (effects (font (size 1.27 1.27)) hide)
     )
@@
     (pin "1")
   )
-  (symbol (lib_id "power:GND") (at 106.68 191.77 0) (unit 1)
+  (symbol (lib_id "power:GND") (at 106.68 194.31 0) (unit 1)
     (in_bom yes) (on_board yes) (fields_autoplaced)
-    (property "Reference" "#PWR0123" (id 0) (at 106.68 198.12 0)
-      (effects (font (size 1.27 1.27)) hide)
-    )
-    (property "Value" "GND" (id 1) (at 106.68 196.85 0))
-    (property "Footprint" "" (id 2) (at 106.68 191.77 0)
-      (effects (font (size 1.27 1.27)) hide)
-    )
-    (property "Datasheet" "" (id 3) (at 106.68 191.77 0)
+    (property "Reference" "#PWR0123" (id 0) (at 106.68 200.66 0)
+      (effects (font (size 1.27 1.27)) hide)
+    )
+    (property "Value" "GND" (id 1) (at 106.68 199.39 0))
+    (property "Footprint" "" (id 2) (at 106.68 194.31 0)
+      (effects (font (size 1.27 1.27)) hide)
+    )
+    (property "Datasheet" "" (id 3) (at 106.68 194.31 0)
       (effects (font (size 1.27 1.27)) hide)
     )
@@
   (symbol (lib_id "power:GND") (at 140.97 193.04 0) (unit 1)
     (in_bom yes) (on_board yes) (fields_autoplaced)
-    (property "Reference" "#PWR?" (id 0) (at 140.97 199.39 0)
+    (property "Reference" "#PWR0115" (id 0) (at 140.97 199.39 0)
       (effects (font (size 1.27 1.27)) hide)
     )
@@
   (symbol (lib_id "Device:R") (at 140.97 189.23 0) (unit 1)
     (in_bom yes) (on_board yes) (fields_autoplaced)
-    (property "Reference" "R?" (id 0) (at 143.51 187.9599 0)
+    (property "Reference" "R35" (id 0) (at 143.51 187.9599 0)
       (effects (font (size 1.27 1.27)) (justify left))
     )
@@
   (symbol (lib_id "ecafe-racer:LED_Green") (at 140.97 181.61 90) (unit 1)
     (in_bom yes) (on_board yes) (fields_autoplaced)
-    (property "Reference" "D?" (id 0) (at 144.78 180.5304 90)
+    (property "Reference" "D20" (id 0) (at 144.78 180.5304 90)
       (effects (font (size 1.27 1.27)) (justify right))
     )
@@
       (reference "#PWR0114") (unit 1) (value "GND") (footprint "")
     )
+    (path "/57522df6-13d5-49b6-b736-3650cb049fbf"
+      (reference "#PWR0115") (unit 1) (value "GND") (footprint "")
+    )
     (path "/8ab74ef5-80a9-48a4-b388-3107db361fe8/51b533c9-c9cf-4b20-956a-5b9c38cb2296"
       (reference "#PWR0116") (unit 1) (value "+3.3V") (footprint "")
@@
       (reference "#PWR0199") (unit 1) (value "+5V") (footprint "")
     )
-    (path "/57522df6-13d5-49b6-b736-3650cb049fbf"
-      (reference "#PWR?") (unit 1) (value "GND") (footprint "")
-    )
     (path "/19c8499b-69ca-41a4-81d4-1e5248b15d37/eeb646f8-ecd2-4f7a-a6bd-d4a25607ff16"
       (reference "BT1") (unit 1) (value "Battery_Cell") (footprint "Battery:BatteryHolder_Keystone_3001_1x12mm")
@@
     )
     (path "/c9ff74f8-0bc9-4f11-a548-132fe582a2f8"
-      (reference "D?") (unit 1) (value "LED_Green") (footprint "LED_SMD:LED_0805_2012Metric_Pad1.15x1.40mm_HandSolder")
+      (reference "D20") (unit 1) (value "LED_Green") (footprint "LED_SMD:LED_0805_2012Metric_Pad1.15x1.40mm_HandSolder")
     )
     (path "/56031da0-b30d-40e7-9bf7-184fa400b03d"
@@
     )
     (path "/802cfdee-6aab-4737-871d-9f7e3f99c57a"
-      (reference "R?") (unit 1) (value "R") (footprint "Resistor_SMD:R_0805_2012Metric")
+      (reference "R35") (unit 1) (value "R") (footprint "Resistor_SMD:R_0805_2012Metric")
     )
     (path "/a37aae83-17bc-4ab3-8207-20408c46a8d9/ce1e3873-ad4a-46e4-bc8e-1516017c2b73"

Commit message: geographical reannotate
Parts:
- removed H4: MountingHole_Pad, MountingHole:MountingHole_3.2mm_M3, symbol Mechanical:MountingHole_Pad
- renumbered D16 to D1, D5 to D16, D18 to D17, D7 to D18, D20 to D2, H3 to H1, H1 to H3, J4 to J2, J3 to J4, J14 to J5, J11 to J6, Q6 to Q2, Q5 to Q3, R24 to R2, R35 to R20, R23 to R3, R30 to R33, R21 to R5, R22 to R7
Connections:
- no-connect marks 4 -> 3
