File: BikeMan.kicad_sch (KiCad schematic)
At the start: 20 parts, among them J2 MicroUSB, J4 Conn_01x06_Male, J5 PushConnector_8pos, J6 PushConnector_8pos, Q2 DMN62D0U-7, Q3 DMN62D0U-7

Commit message: added test points and cleaned up silk screen
Parts:
- added TP? (x4): TestPoint, TestPoint:TestPoint_Pad_D1.5mm, symbol Connector:TestPoint
Connections:
- net SCL_{3.3V}: now also TP?.1
- net SDA_{3.3V}: now also TP?.1
- net USB.+: now also TP?.1
- net USB.-: now also TP?.1
Changed lines of the file:
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@@
+    (stroke (width 0) (type solid) (color 0 0 0 0))
+  )
+  (wire (pts (xy 187.96 154.94) (xy 196.85 154.94))
+    (stroke (width 0) (type solid) (color 0 0 0 0))
+  )
+  (wire (pts (xy 187.96 157.48) (xy 196.85 157.48))
+    (stroke (width 0) (type solid) (color 0 0 0 0))
+  )
+  (wire (pts (xy 187.96 160.02) (xy 196.85 160.02))
+    (stroke (width 0) (type solid) (color 0 0 0 0))
+  )
+  (wire (pts (xy 187.96 162.56) (xy 196.85 162.56))
     (stroke (width 0) (type solid) (color 0 0 0 0))
   )
@@
   (label "SCL_{5V}" (at 184.15 111.76 180)
     (effects (font (size 1.27 1.27)) (justify right bottom))
+  )
+  (label "SDA_{3.3V}" (at 187.96 154.94 0)
+    (effects (font (size 1.27 1.27)) (justify left bottom))
+  )
+  (label "SCL_{3.3V}" (at 187.96 157.48 0)
+    (effects (font (size 1.27 1.27)) (justify left bottom))
+  )
+  (label "USB.+" (at 187.96 160.02 0)
+    (effects (font (size 1.27 1.27)) (justify left bottom))
+  )
+  (label "USB.-" (at 187.96 162.56 0)
+    (effects (font (size 1.27 1.27)) (justify left bottom))
   )
   (label "CAN_{H}" (at 218.44 31.75 180)
@@
     )
     (property "Datasheet" "" (id 3) (at 107.95 171.45 0)
+      (effects (font (size 1.27 1.27)) hide)
+    )
+    (pin "1")
+  )
+  (symbol (lib_id "Connector:TestPoint") (at 196.85 154.94 270) (unit 1)
+    (in_bom yes) (on_board yes)
+    (property "Reference" "TP?" (id 0) (at 202.3809 155.0671 90)
+      (effects (font (size 1.27 1.27)) (justify left))
+    )
+    (property "Value" "TestPoint" (id 1) (at 197.542 156.337 0)
+      (effects (font (size 1.27 1.27)) (justify left) hide)
+    )
+    (property "Footprint" "TestPoint:TestPoint_Pad_D1.5mm" (id 2) (at 196.85 160.02 0)
+      (effects (font (size 1.27 1.27)) hide)
+    )
+    (property "Datasheet" "~" (id 3) (at 196.85 160.02 0)
+      (effects (font (size 1.27 1.27)) hide)
+    )
+    (pin "1")
+  )
+  (symbol (lib_id "Connector:TestPoint") (at 196.85 157.48 270) (unit 1)
+    (in_bom yes) (on_board yes)
+    (property "Reference" "TP?" (id 0) (at 202.3809 157.6071 90)
+      (effects (font (size 1.27 1.27)) (justify left))
+    )
+    (property "Value" "TestPoint" (id 1) (at 197.542 158.877 0)
+      (effects (font (size 1.27 1.27)) (justify left) hide)
+    )
+    (property "Footprint" "TestPoint:TestPoint_Pad_D1.5mm" (id 2) (at 196.85 162.56 0)
+      (effects (font (size 1.27 1.27)) hide)
+    )
+    (property "Datasheet" "~" (id 3) (at 196.85 162.56 0)
+      (effects (font (size 1.27 1.27)) hide)
+    )
+    (pin "1")
+  )
+  (symbol (lib_id "Connector:TestPoint") (at 196.85 160.02 270) (unit 1)
+    (in_bom yes) (on_board yes)
+    (property "Reference" "TP?" (id 0) (at 202.3809 160.1471 90)
+      (effects (font (size 1.27 1.27)) (justify left))
+    )
+    (property "Value" "TestPoint" (id 1) (at 197.542 161.417 0)
+      (effects (font (size 1.27 1.27)) (justify left) hide)
+    )
+    (property "Footprint" "TestPoint:TestPoint_Pad_D1.5mm" (id 2) (at 196.85 165.1 0)
+      (effects (font (size 1.27 1.27)) hide)
+    )
+    (property "Datasheet" "~" (id 3) (at 196.85 165.1 0)
+      (effects (font (size 1.27 1.27)) hide)
+    )
+    (pin "1")
+  )
+  (symbol (lib_id "Connector:TestPoint") (at 196.85 162.56 270) (unit 1)
+    (in_bom yes) (on_board yes)
+    (property "Reference" "TP?" (id 0) (at 202.3809 162.6871 90)
+      (effects (font (size 1.27 1.27)) (justify left))
+    )
+    (property "Value" "TestPoint" (id 1) (at 197.542 163.957 0)
+      (effects (font (size 1.27 1.27)) (justify left) hide)
+    )
+    (property "Footprint" "TestPoint:TestPoint_Pad_D1.5mm" (id 2) (at 196.85 167.64 0)
+      (effects (font (size 1.27 1.27)) hide)
+    )
+    (property "Datasheet" "~" (id 3) (at 196.85 167.64 0)
       (effects (font (size 1.27 1.27)) hide)
     )
@@
       (reference "#PWR0149") (unit 1) (value "GND") (footprint "")
     )
+    (path "/97a6e0d0-e45e-4fe9-a578-968187c50165/e96064e2-a177-4e8b-80a5-c826e98ca808"
+      (reference "#PWR0150") (unit 1) (value "GND") (footprint "")
+    )
+    (path "/97a6e0d0-e45e-4fe9-a578-968187c50165/2550d342-2a9b-4dc8-96d5-7431fa5449a0"
+      (reference "#PWR0151") (unit 1) (value "+12V") (footprint "")
+    )
+    (path "/97a6e0d0-e45e-4fe9-a578-968187c50165/45143c1b-1953-4f38-a51d-98a350b9ba7a"
+      (reference "#PWR0152") (unit 1) (value "+3.3V") (footprint "")
+    )
     (path "/97a6e0d0-e45e-4fe9-a578-968187c50165/fcb0cd51-9f00-497e-9bbc-b2dbab7db47b"
       (reference "#PWR0155") (unit 1) (value "GND") (footprint "")
@@
       (reference "TP8") (unit 1) (value "TestPoint") (footprint "TestPoint:TestPoint_Pad_D1.5mm")
     )
+    (path "/97a6e0d0-e45e-4fe9-a578-968187c50165/2d418802-792c-4bff-a16f-9bfd29b1feee"
+      (reference "TP9") (unit 1) (value "TestPoint") (footprint "TestPoint:TestPoint_Pad_D1.5mm")
+    )
+    (path "/97a6e0d0-e45e-4fe9-a578-968187c50165/898de7a0-3721-4553-9f98-66900118b4a7"
+      (reference "TP10") (unit 1) (value "TestPoint") (footprint "TestPoint:TestPoint_Pad_D1.5mm")
+    )
+    (path "/97a6e0d0-e45e-4fe9-a578-968187c50165/d3efffdd-e65e-43fc-86e9-e74de7d387ad"
+      (reference "TP11") (unit 1) (value "TestPoint") (footprint "TestPoint:TestPoint_Pad_D1.5mm")
+    )
+    (path "/97a6e0d0-e45e-4fe9-a578-968187c50165/54bd8716-8ab8-45cd-84e9-0c54e9a07508"
+      (reference "TP12") (unit 1) (value "TestPoint") (footprint "TestPoint:TestPoint_Pad_D1.5mm")
+    )
+    (path "/97a6e0d0-e45e-4fe9-a578-968187c50165/f8c4df60-e461-4b0f-98d9-c07d60ac5b7c"
+      (reference "TP13") (unit 1) (value "TestPoint") (footprint "TestPoint:TestPoint_Pad_D1.5mm")
+    )
+    (path "/0086bb93-d03e-4eea-8c03-1dbf6e657c05"
+      (reference "TP?") (unit 1) (value "TestPoint") (footprint "TestPoint:TestPoint_Pad_D1.5mm")
+    )
+    (path "/e43f27d1-1967-472c-a6a2-b0a41cccd019"
+      (reference "TP?") (unit 1) (value "TestPoint") (footprint "TestPoint:TestPoint_Pad_D1.5mm")
+    )
+    (path "/e5b894f5-b6f6-4404-b031-711072bdbe57"
+      (reference "TP?") (unit 1) (value "TestPoint") (footprint "TestPoint:TestPoint_Pad_D1.5mm")
+    )
+    (path "/f14a962c-1b9d-46a0-8cc1-8946d723b862"
+      (reference "TP?") (unit 1) (value "TestPoint") (footprint "TestPoint:TestPoint_Pad_D1.5mm")
+    )
     (path "/8ab74ef5-80a9-48a4-b388-3107db361fe8/b6568ad9-8100-4e5f-ad69-cce5b5be4e99"

Commit message: updated 3d models
Parts:
- J5: footprint footprints:CUI_TBL004-508-08BE-2BE -> ecafe-racer:CUI_TBL004-508-08BE-2BE; symbol symbols:PushConnector_8pos -> ecafe-racer:PushConnector_8pos
- gave numbers to parts that had none: 4
Changed lines of the file:
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@@
   (symbol (lib_id "Connector:TestPoint") (at 196.85 154.94 270) (unit 1)
     (in_bom yes) (on_board yes)
-    (property "Reference" "TP?" (id 0) (at 202.3809 155.0671 90)
+    (property "Reference" "TP14" (id 0) (at 202.3809 155.0671 90)
       (effects (font (size 1.27 1.27)) (justify left))
     )
@@
   (symbol (lib_id "Connector:TestPoint") (at 196.85 157.48 270) (unit 1)
     (in_bom yes) (on_board yes)
-    (property "Reference" "TP?" (id 0) (at 202.3809 157.6071 90)
+    (property "Reference" "TP15" (id 0) (at 202.3809 157.6071 90)
       (effects (font (size 1.27 1.27)) (justify left))
     )
@@
   (symbol (lib_id "Connector:TestPoint") (at 196.85 160.02 270) (unit 1)
     (in_bom yes) (on_board yes)
-    (property "Reference" "TP?" (id 0) (at 202.3809 160.1471 90)
+    (property "Reference" "TP16" (id 0) (at 202.3809 160.1471 90)
       (effects (font (size 1.27 1.27)) (justify left))
     )
@@
   (symbol (lib_id "Connector:TestPoint") (at 196.85 162.56 270) (unit 1)
     (in_bom yes) (on_board yes)
-    (property "Reference" "TP?" (id 0) (at 202.3809 162.6871 90)
+    (property "Reference" "TP17" (id 0) (at 202.3809 162.6871 90)
       (effects (font (size 1.27 1.27)) (justify left))
     )
@@
     (pin "6")
   )
-  (symbol (lib_name "symbols:PushConnector_8pos_1") (lib_id "symbols:PushConnector_8pos") (at 242.57 71.12 0) (unit 1)
+  (symbol (lib_id "ecafe-racer:PushConnector_8pos") (at 242.57 71.12 0) (unit 1)
     (in_bom yes) (on_board yes)
     (property "Reference" "J5" (id 0) (at 247.0913 78.0478 0)
@@
       (effects (font (size 1.27 1.27)) (justify left) hide)
     )
-    (property "Footprint" "footprints:CUI_TBL004-508-08BE-2BE" (id 2) (at 242.57 71.12 0)
+    (property "Footprint" "ecafe-racer:CUI_TBL004-508-08BE-2BE" (id 2) (at 242.57 71.12 0)
       (effects (font (size 1.27 1.27)) hide)
     )
@@
     )
     (path "/af553289-cbab-4153-b69b-747ee91d5403"
-      (reference "J5") (unit 1) (value "PushConnector_8pos") (footprint "footprints:CUI_TBL004-508-08BE-2BE")
+      (reference "J5") (unit 1) (value "PushConnector_8pos") (footprint "ecafe-racer:CUI_TBL004-508-08BE-2BE")
     )
     (path "/a89789bf-aae5-4f10-97fc-c73c3ffe195f"
@@
     )
     (path "/0086bb93-d03e-4eea-8c03-1dbf6e657c05"
-      (reference "TP?") (unit 1) (value "TestPoint") (footprint "TestPoint:TestPoint_Pad_D1.5mm")
+      (reference "TP14") (unit 1) (value "TestPoint") (footprint "TestPoint:TestPoint_Pad_D1.5mm")
+    )
+    (path "/f14a962c-1b9d-46a0-8cc1-8946d723b862"
+      (reference "TP15") (unit 1) (value "TestPoint") (footprint "TestPoint:TestPoint_Pad_D1.5mm")
     )
     (path "/e43f27d1-1967-472c-a6a2-b0a41cccd019"
-      (reference "TP?") (unit 1) (value "TestPoint") (footprint "TestPoint:TestPoint_Pad_D1.5mm")
+      (reference "TP16") (unit 1) (value "TestPoint") (footprint "TestPoint:TestPoint_Pad_D1.5mm")
     )
     (path "/e5b894f5-b6f6-4404-b031-711072bdbe57"
-      (reference "TP?") (unit 1) (value "TestPoint") (footprint "TestPoint:TestPoint_Pad_D1.5mm")
-    )
-    (path "/f14a962c-1b9d-46a0-8cc1-8946d723b862"
-      (reference "TP?") (unit 1) (value "TestPoint") (footprint "TestPoint:TestPoint_Pad_D1.5mm")
+      (reference "TP17") (unit 1) (value "TestPoint") (footprint "TestPoint:TestPoint_Pad_D1.5mm")
     )
     (path "/8ab74ef5-80a9-48a4-b388-3107db361fe8/b6568ad9-8100-4e5f-ad69-cce5b5be4e99"
